File: KiCad PCBs/Master Shield/Master Shield.kicad_pcb (KiCad board)
At the start: 2 copper layers, 78.8 x 53.3 mm, 32 parts, among them J1 Power, J2 PWM, J3 Communication

Commit message: Final Master Shield files
Other:
- rule pad_to_mask_clearance: 0.0508 -> 0
- board text added: "DCS-BIOS RS485 Triple Master Rev. 1"
- board text removed: "RS485 Triple Master Rev. 1"
Changed lines of the file:
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@@
       (layer "B.Paste" (type "Bottom Solder Paste"))
       (layer "B.SilkS" (type "Bottom Silk Screen"))
-      (copper_finish "None")
+      (copper_finish "ENIG")
       (dielectric_constraints no)
     )
-    (pad_to_mask_clearance 0.0508)
-    (solder_mask_min_width 0.101)
+    (pad_to_mask_clearance 0)
     (aux_axis_origin 100 100)
     (pcbplotparams
@@
     (descr "Resistor SMD 0805 (2012 Metric), square (rectangular) end terminal, IPC_7351 nominal, (Body size source: IPC-SM-782 page 72, https://www.pcb-3d.com/wordpress/wp-content/uploads/ipc-sm-782a_amendment_1_and_2.pdf), generated with kicad-footprint-generator")
     (tags "resistor")
+    (property "LCSC" "C17437")
     (property "Sheetfile" "Master Shield.kicad_sch")
     (property "Sheetname" "")
@@
     (descr "SOIC-8_L5.0-W4.0-P1.27-LS6.0-BL footprint")
     (tags "SOIC-8_L5.0-W4.0-P1.27-LS6.0-BL footprint")
+    (property "LCSC" "C9953")
     (property "Sheetfile" "Master Shield.kicad_sch")
     (property "Sheetname" "")
@@
     (descr "Resistor SMD 0805 (2012 Metric), square (rectangular) end terminal, IPC_7351 nominal, (Body size source: IPC-SM-782 page 72, https://www.pcb-3d.com/wordpress/wp-content/uploads/ipc-sm-782a_amendment_1_and_2.pdf), generated with kicad-footprint-generator")
     (tags "resistor")
+    (property "LCSC" "C17398")
     (property "Sheetfile" "Master Shield.kicad_sch")
     (property "Sheetname" "")
@@
     (property "Sheetfile" "Master Shield.kicad_sch")
     (property "Sheetname" "")
-    (attr through_hole)
+    (property "exclude_from_bom" "")
+    (attr through_hole exclude_from_bom)
     (fp_text reference "PSU1" (at 0 -8.148717 90) (layer "F.SilkS")
       (effects (font (size 1 1) (thickness 0.15)))
@@
     (descr "LED SMD 0603 (1608 Metric), square (rectangular) end terminal, IPC_7351 nominal, (Body size source: http://www.tortai-tech.com/upload/download/2011102023233369053.pdf), generated with kicad-footprint-generator")
     (tags "LED")
+    (property "LCSC" "C72041")
     (property "Sheetfile" "Master Shield.kicad_sch")
     (property "Sheetname" "")
@@
     (descr "CONN-TH_430450812 footprint")
     (tags "CONN-TH_430450812 footprint")
+    (property "LCSC" "C277661")
     (property "Sheetfile" "Master Shield.kicad_sch")
     (property "Sheetname" "")
@@
     (descr "C0402 footprint")
     (tags "C0402 footprint")
+    (property "LCSC" "C1525")
     (property "Sheetfile" "Master Shield.kicad_sch")
     (property "Sheetname" "")
@@
     (descr "C0402 footprint")
     (tags "C0402 footprint")
+    (property "LCSC" "C1525")
     (property "Sheetfile" "Master Shield.kicad_sch")
     (property "Sheetname" "")
@@
     (descr "Resistor SMD 0805 (2012 Metric), square (rectangular) end terminal, IPC_7351 nominal, (Body size source: IPC-SM-782 page 72, https://www.pcb-3d.com/wordpress/wp-content/uploads/ipc-sm-782a_amendment_1_and_2.pdf), generated with kicad-footprint-generator")
     (tags "resistor")
+    (property "LCSC" "C17398")
     (property "Sheetfile" "Master Shield.kicad_sch")
     (property "Sheetname" "")
@@
     (descr "SOIC-8_L5.0-W4.0-P1.27-LS6.0-BL footprint")
     (tags "SOIC-8_L5.0-W4.0-P1.27-LS6.0-BL footprint")
+    (property "LCSC" "C9953")
     (property "Sheetfile" "Master Shield.kicad_sch")
     (property "Sheetname" "")
@@
     (descr "LED SMD 0603 (1608 Metric), square (rectangular) end terminal, IPC_7351 nominal, (Body size source: http://www.tortai-tech.com/upload/download/2011102023233369053.pdf), generated with kicad-footprint-generator")
     (tags "LED")
+    (property "LCSC" "C72041")
     (property "Sheetfile" "Master Shield.kicad_sch")
     (property "Sheetname" "")
@@
     (descr "LED SMD 0603 (1608 Metric), square (rectangular) end terminal, IPC_7351 nominal, (Body size source: http://www.tortai-tech.com/upload/download/2011102023233369053.pdf), generated with kicad-footprint-generator")
     (tags "LED")
+    (property "LCSC" "C72041")
     (property "Sheetfile" "Master Shield.kicad_sch")
     (property "Sheetname" "")
@@
     (property "Sheetfile" "Master Shield.kicad_sch")
     (property "Sheetname" "")
-    (attr through_hole)
+    (property "exclude_from_bom" "")
+    (attr through_hole exclude_from_bom)
     (fp_text reference "PSU3" (at 0 -8.148717 90) (layer "F.SilkS")
       (effects (font (size 1 1) (thickness 0.15)))
@@
     (descr "LED SMD 0603 (1608 Metric), square (rectangular) end terminal, IPC_7351 nominal, (Body size source: http://www.tortai-tech.com/upload/download/2011102023233369053.pdf), generated with kicad-footprint-generator")
     (tags "LED")
-    (property "Field4" "5V")
+    (property "LCSC" "C72041")
     (property "Sheetfile" "Master Shield.kicad_sch")
     (property "Sheetname" "")
@@
     (property "Sheetfile" "Master Shield.kicad_sch")
     (property "Sheetname" "")
-    (attr through_hole)
+    (property "exclude_from_bom" "")
+    (attr through_hole exclude_from_bom)
     (fp_text reference "PSU2" (at 0 -8.148717 90) (layer "F.SilkS")
       (effects (font (size 1 1) (thickness 0.15)))
@@
     (descr "C0402 footprint")
     (tags "C0402 footprint")
+    (property "LCSC" "C1525")
     (property "Sheetfile" "Master Shield.kicad_sch")
     (property "Sheetname" "")
@@
     (descr "Resistor SMD 0805 (2012 Metric), square (rectangular) end terminal, IPC_7351 nominal, (Body size source: IPC-SM-782 page 72, https://www.pcb-3d.com/wordpress/wp-content/uploads/ipc-sm-782a_amendment_1_and_2.pdf), generated with kicad-footprint-generator")
     (tags "resistor")
+    (property "LCSC" "C17398")
     (property "Sheetfile" "Master Shield.kicad_sch")
     (property "Sheetname" "")
@@
     (descr "Resistor SMD 0805 (2012 Metric), square (rectangular) end terminal, IPC_7351 nominal, (Body size source: IPC-SM-782 page 72, https://www.pcb-3d.com/wordpress/wp-content/uploads/ipc-sm-782a_amendment_1_and_2.pdf), generated with kicad-footprint-generator")
     (tags "resistor")
+    (property "LCSC" "C17655")
     (property "Sheetfile" "Master Shield.kicad_sch")
     (property "Sheetname" "")
@@
     (property "Sheetfile" "Master Shield.kicad_sch")
     (property "Sheetname" "")
-    (attr through_hole)
+    (property "exclude_from_bom" "")
+    (attr through_hole exclude_from_bom)
     (fp_text reference "F2" (at 8.89 1.27) (layer "F.SilkS")
       (effects (font (size 1 1) (thickness 0.15)))
@@
     (descr "CONN-TH_430450812 footprint")
     (tags "CONN-TH_430450812 footprint")
+    (property "LCSC" "C277661")
     (property "Sheetfile" "Master Shield.kicad_sch")
     (property "Sheetname" "")
@@
     (descr "SOIC-8_L5.0-W4.0-P1.27-LS6.0-BL footprint")
     (tags "SOIC-8_L5.0-W4.0-P1.27-LS6.0-BL footprint")
+    (property "LCSC" "C9953")
     (property "Sheetfile" "Master Shield.kicad_sch")
     (property "Sheetname" "")
@@
     (descr "Resistor SMD 0805 (2012 Metric), square (rectangular) end terminal, IPC_7351 nominal, (Body size source: IPC-SM-782 page 72, https://www.pcb-3d.com/wordpress/wp-content/uploads/ipc-sm-782a_amendment_1_and_2.pdf), generated with kicad-footprint-generator")
     (tags "resistor")
+    (property "LCSC" "C17437")
     (property "Sheetfile" "Master Shield.kicad_sch")
     (property "Sheetname" "")
@@
     (property "Sheetfile" "Master Shield.kicad_sch")
     (property "Sheetname" "")
-    (attr through_hole)
+    (property "exclude_from_bom" "")
+    (attr through_hole exclude_from_bom)
     (fp_text reference "F1" (at 8.89 1.27) (layer "F.SilkS")
       (effects (font (size 1 1) (thickness 0.15)))
@@
     (property "Sheetfile" "Master Shield.kicad_sch")
     (property "Sheetname" "")
-    (attr through_hole)
+    (property "exclude_from_bom" "")
+    (attr through_hole exclude_from_bom)
     (fp_text reference "F3" (at 8.89 1.27) (layer "F.SilkS")
       (effects (font (size 1 1) (thickness 0.15)))
@@
     (descr "Resistor SMD 0805 (2012 Metric), square (rectangular) end terminal, IPC_7351 nominal, (Body size source: IPC-SM-782 page 72, https://www.pcb-3d.com/wordpress/wp-content/uploads/ipc-sm-782a_amendment_1_and_2.pdf), generated with kicad-footprint-generator")
     (tags "resistor")
+    (property "LCSC" "C17437")
     (property "Sheetfile" "Master Shield.kicad_sch")
     (property "Sheetname" "")
@@
     (descr "CONN-TH_430450812 footprint")
     (tags "CONN-TH_430450812 footprint")
+    (property "LCSC" "C277661")
     (property "Sheetfile" "Master Shield.kicad_sch")
     (property "Sheetname" "")
@@
     (descr "Through hole straight pin header, 1x08, 2.54mm pitch, single row")
     (tags "Through hole pin header THT 1x08 2.54mm single row")
+    (property "LCSC" "C124381")
     (property "Sheetfile" "Master Shield.kicad_sch")
     (property "Sheetname" "")
@@
     (descr "Through hole straight pin header, 1x08, 2.54mm pitch, single row")
     (tags "Through hole pin header THT 1x08 2.54mm single row")
+    (property "LCSC" "C124381")
     (property "Sheetfile" "Master Shield.kicad_sch")
     (property "Sheetname" "")
@@
     (descr "Through hole straight pin header, 1x08, 2.54mm pitch, single row")
     (tags "Through hole pin header THT 1x08 2.54mm single row")
+    (property "LCSC" "C124381")
     (property "Sheetfile" "Master Shield.kicad_sch")
     (property "Sheetname" "")
@@
     (effects (font (size 0.8128 0.8128) (thickness 0.1016)) (justify right))
   )
-  (gr_text "RS485 Triple Master Rev. 1" (at 127.305 73.33 90) (layer "F.SilkS")
+  (gr_text "DCS-BIOS RS485 Triple Master Rev. 1" (at 127.305 72.39 90) (layer "F.SilkS")
     (effects (font (size 1.5 1.5) (thickness 0.3)))
   )
