File: KiCad PCBs/Slave/Slave.kicad_sch (KiCad schematic)
At the start: 50 parts, among them J1 Screw_Terminal_01x02, J10 AVR-ISP-6, J11 Conn_01x06_Female, J12 Screw_Terminal_01x02, J13 Screw_Terminal_01x02, J14 Screw_Terminal_01x02, J15 Screw_Terminal_01x02, J16 Screw_Terminal_01x02, J2 Screw_Terminal_01x02, J3 Screw_Terminal_01x02, J4 Screw_Terminal_01x02, J5 Screw_Terminal_01x02, J6 Screw_Terminal_01x02, J7 Screw_Terminal_01x02, J8 Screw_Terminal_01x02, J9 Screw_Terminal_01x02, SW1 SW_DIP_x02, SW2 SW_DIP_x02, SW3 SW_MEC_5E, U1 ATmega328P-AU, U2 MAX487ESA+T, U3 ULN2003A, U4 LM358DR2G, U5 AMS1117-5.0, Y1 Crystal_GND24

Commit message: Slave WIP
Parts:
- R5: now left out of the parts list
Connections:
- net +5V: no longer R5.1
- net RESET: no longer R5.2
- no-connect marks 5 -> 8
Other:
- note added: "This resistor is replaced by R3"
- moved on the sheet: R5, SW3
Changed lines of the file:
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@@
   (junction (at 30.48 154.94) (diameter 0) (color 0 0 0 0)
   )
+  (no_connect (at 48.26 22.86))
   (no_connect (at 133.35 69.85))
   (no_connect (at 133.35 72.39))
@@
   (no_connect (at 275.59 93.98))
   (no_connect (at 255.27 93.98))
+  (no_connect (at 48.26 33.02))
+  (no_connect (at 48.26 25.4))
   (wire (pts (xy 168.91 82.55) (xy 166.37 82.55))
     (stroke (width 0) (type default) (color 0 0 0 0))
@@
     (stroke (width 0) (type default) (color 0 0 0 0))
   )
-  (wire (pts (xy 26.67 38.1) (xy 29.21 38.1))
+  (wire (pts (xy 25.4 35.56) (xy 27.94 35.56))
     (stroke (width 0) (type default) (color 0 0 0 0))
   )
@@
     (stroke (width 0) (type default) (color 0 0 0 0))
   )
-  (wire (pts (xy 49.53 25.4) (xy 49.53 27.94))
-    (stroke (width 0) (type default) (color 0 0 0 0))
-  )
   (wire (pts (xy 43.18 137.16) (xy 43.18 139.7))
     (stroke (width 0) (type default) (color 0 0 0 0))
@@
     (stroke (width 0) (type default) (color 0 0 0 0))
   )
-  (wire (pts (xy 49.53 35.56) (xy 49.53 38.1))
-    (stroke (width 0) (type default) (color 0 0 0 0))
-  )
   (wire (pts (xy 25.4 101.6) (xy 25.4 106.68))
     (stroke (width 0) (type default) (color 0 0 0 0))
@@
     (stroke (width 0) (type default) (color 0 0 0 0))
   )
+  (wire (pts (xy 48.26 35.56) (xy 48.26 38.1))
+    (stroke (width 0) (type default) (color 0 0 0 0))
+  )
   (wire (pts (xy 38.1 119.38) (xy 38.1 121.92))
     (stroke (width 0) (type default) (color 0 0 0 0))
@@
     (stroke (width 0) (type default) (color 0 0 0 0))
   )
-  (wire (pts (xy 39.37 38.1) (xy 49.53 38.1))
+  (wire (pts (xy 38.1 35.56) (xy 48.26 35.56))
     (stroke (width 0) (type default) (color 0 0 0 0))
   )
@@
     (effects (font (size 1.27 1.27)) (justify left bottom))
   )
-  (label "RESET" (at 41.91 38.1 0)
-    (effects (font (size 1.27 1.27)) (justify left bottom))
+  (text "This resistor is replaced by R3" (at 45.72 33.02 90)
+    (effects (font (size 0.54 0.54)) (justify left bottom))
   )
   (global_label "A1" (shape input) (at 168.91 90.17 0) (fields_autoplaced)
@@
     )
   )
+  (global_label "RESET" (shape output) (at 48.26 38.1 270) (fields_autoplaced)
+    (effects (font (size 1.27 1.27)) (justify right))
+    (property "Intersheet References" "${INTERSHEET_REFS}" (id 0) (at 48.3394 46.2583 90)
+      (effects (font (size 1.27 1.27)) (justify right) hide)
+    )
+  )
   (global_label "TXD" (shape input) (at 194.31 40.64 180) (fields_autoplaced)
     (effects (font (size 1.27 1.27)) (justify right))
@@
   (symbol (lib_id "power:+12V") (at 21.59 60.96 90) (unit 1)
     (in_bom yes) (on_board yes) (fields_autoplaced)
-    (property "Reference" "#PWR?" (id 0) (at 25.4 60.96 0)
+    (property "Reference" "#PWR0103" (id 0) (at 25.4 60.96 0)
       (effects (font (size 1.27 1.27)) hide)
     )
@@
     (pin "1")
   )
-  (symbol (lib_id "power:+5V") (at 49.53 25.4 0) (unit 1)
+  (symbol (lib_id "power:+5V") (at 48.26 22.86 0) (unit 1)
     (in_bom yes) (on_board yes) (fields_autoplaced)
-    (property "Reference" "#PWR0105" (id 0) (at 49.53 29.21 0)
+    (property "Reference" "#PWR0105" (id 0) (at 48.26 26.67 0)
       (effects (font (size 1.27 1.27)) hide)
     )
-    (property "Value" "+5V" (id 1) (at 49.53 20.32 0))
-    (property "Footprint" "" (id 2) (at 49.53 25.4 0)
+    (property "Value" "+5V" (id 1) (at 48.26 17.78 0))
+    (property "Footprint" "" (id 2) (at 48.26 22.86 0)
       (effects (font (size 1.27 1.27)) hide)
     )
-    (property "Datasheet" "" (id 3) (at 49.53 25.4 0)
+    (property "Datasheet" "" (id 3) (at 48.26 22.86 0)
       (effects (font (size 1.27 1.27)) hide)
     )
@@
     (pin "2")
   )
-  (symbol (lib_id "Device:R") (at 49.53 31.75 0) (unit 1)
-    (in_bom yes) (on_board yes) (fields_autoplaced)
-    (property "Reference" "R5" (id 0) (at 52.07 30.4799 0)
+  (symbol (lib_id "Device:R") (at 48.26 29.21 0) (unit 1)
+    (in_bom no) (on_board no) (fields_autoplaced)
+    (property "Reference" "R5" (id 0) (at 50.8 27.9399 0)
       (effects (font (size 1.27 1.27)) (justify left))
     )
-    (property "Value" "1K" (id 1) (at 52.07 33.0199 0)
+    (property "Value" "1K" (id 1) (at 50.8 30.4799 0)
       (effects (font (size 1.27 1.27)) (justify left))
     )
-    (property "Footprint" "Resistor_SMD:R_0402_1005Metric" (id 2) (at 47.752 31.75 90)
+    (property "Footprint" "Resistor_SMD:R_0402_1005Metric" (id 2) (at 46.482 29.21 90)
       (effects (font (size 1.27 1.27)) hide)
     )
-    (property "Datasheet" "~" (id 3) (at 49.53 31.75 0)
+    (property "Datasheet" "~" (id 3) (at 48.26 29.21 0)
       (effects (font (size 1.27 1.27)) hide)
     )
@@
     (pin "2")
   )
-  (symbol (lib_id "power:GND") (at 26.67 38.1 0) (unit 1)
+  (symbol (lib_id "power:GND") (at 25.4 35.56 0) (unit 1)
     (in_bom yes) (on_board yes)
-    (property "Reference" "#PWR0104" (id 0) (at 26.67 44.45 0)
+    (property "Reference" "#PWR0104" (id 0) (at 25.4 41.91 0)
       (effects (font (size 1.27 1.27)) hide)
     )
-    (property "Value" "GND" (id 1) (at 26.67 43.18 0))
-    (property "Footprint" "" (id 2) (at 26.67 38.1 0)
+    (property "Value" "GND" (id 1) (at 25.4 40.64 0))
+    (property "Footprint" "" (id 2) (at 25.4 35.56 0)
       (effects (font (size 1.27 1.27)) hide)
     )
-    (property "Datasheet" "" (id 3) (at 26.67 38.1 0)
+    (property "Datasheet" "" (id 3) (at 25.4 35.56 0)
       (effects (font (size 1.27 1.27)) hide)
     )
@@
     (pin "1")
   )
-  (symbol (lib_id "Switch:SW_MEC_5E") (at 34.29 38.1 0) (unit 1)
+  (symbol (lib_id "Switch:SW_MEC_5E") (at 33.02 35.56 0) (unit 1)
     (in_bom yes) (on_board yes) (fields_autoplaced)
-    (property "Reference" "SW3" (id 0) (at 34.29 30.48 0))
-    (property "Value" "SW_MEC_5E" (id 1) (at 34.29 30.48 0)
+    (property "Reference" "SW3" (id 0) (at 33.02 27.94 0))
+    (property "Value" "SW_MEC_5E" (id 1) (at 33.02 27.94 0)
       (effects (font (size 1.27 1.27)) hide)
     )
-    (property "Footprint" "A10 KiCad Libraries:SW-SMD_4P-L5.1-W5.1-P3.70-LS6.5-TL-2" (id 2) (at 34.29 30.48 0)
+    (property "Footprint" "A10 KiCad Libraries:SW-SMD_4P-L5.1-W5.1-P3.70-LS6.5-TL-2" (id 2) (at 33.02 27.94 0)
       (effects (font (size 1.27 1.27)) hide)
     )
-    (property "Datasheet" "http://www.apem.com/int/index.php?controller=attachment&id_attachment=1371" (id 3) (at 34.29 30.48 0)
+    (property "Datasheet" "http://www.apem.com/int/index.php?controller=attachment&id_attachment=1371" (id 3) (at 33.02 27.94 0)
       (effects (font (size 1.27 1.27)) hide)
     )
@@
       (reference "#PWR0102") (unit 1) (value "GND") (footprint "")
     )
+    (path "/1d7d13da-6155-4f5e-b055-b0667fd2dc2b"
+      (reference "#PWR0103") (unit 1) (value "+12V") (footprint "")
+    )
     (path "/bca02340-bac0-4826-b369-7dfd2dbaae17"
       (reference "#PWR0104") (unit 1) (value "GND") (footprint "")
@@
       (reference "#PWR0146") (unit 1) (value "+5V") (footprint "")
     )
-    (path "/1d7d13da-6155-4f5e-b055-b0667fd2dc2b"
-      (reference "#PWR?") (unit 1) (value "+12V") (footprint "")
-    )
     (path "/df5accf7-095f-40f9-b40a-a9b9e4c1a11a"

Commit message: Slave WIP
Parts:
- removed D3, D4: D, A10 KiCad Libraries:SOD-123F_L2.8-W1.8-LS3.7-RD, symbol Device:D
- removed U4: LM358DR2G, Package_SO:SOIC-8_3.9x4.9mm_P1.27mm, symbol Amplifier_Operational:LM358
- added R10, R9: 1.8K, Resistor_SMD:R_0805_2012Metric, symbol Device:R
- R7, R8: value 1K -> 1.8K; footprint Resistor_SMD:R_0402_1005Metric -> Resistor_SMD:R_0805_2012Metric
Connections:
- net +5V: no longer R7.2, RJ1.1
- net RXD: now also R7.2, R9.2
- net TXD: now also R8.2, R10.2
- net ACT: no longer names the net of RJ1.2
- net ACT: now also R10.1; no longer R8.2
- new net: R9.1, RJ1.1
Other:
- note removed: "Activity LEDs"
- note removed: "Connects via TP cable to activity LED in Hub"

Commit message: Slave WIP
Parts:
- C1: LCSC (none) -> C1779
- C10: LCSC (none) -> C15525
- C11, C2, C3, C4, C6: LCSC (none) -> C52923
- C5, C7: LCSC (none) -> C1525
- C8, C9: value 16pF -> 15pF; LCSC (none) -> C1548
- D1, D2: LCSC (none) -> C72041
- D5: LCSC (none) -> C81598
- J1, J12, J13, J14, J15, J16, J2, J3, J4, J5, J6, J7, J8, J9: LCSC (none) -> C8404
- J10: LCSC (none) -> C492420
- J11: LCSC (none) -> C40877
- R1, R2, R4, R5: footprint Resistor_SMD:R_0402_1005Metric -> Resistor_SMD:R_0805_2012Metric; LCSC (none) -> C17513
- R10, R7, R8, R9: LCSC (none) -> C17398
- R3: footprint Resistor_SMD:R_0402_1005Metric -> Resistor_SMD:R_0805_2012Metric; LCSC (none) -> C17414
- R6: footprint Resistor_SMD:R_0402_1005Metric -> Resistor_SMD:R_0805_2012Metric; LCSC (none) -> C17437
- SW1, SW2: LCSC (none) -> C367376
- SW3: LCSC (none) -> C318884
- U1: LCSC (none) -> C14877
- U2: LCSC (none) -> C9953
- U3: LCSC (none) -> C7512
- U5: LCSC (none) -> C6187
- Y1: LCSC (none) -> C13738
Connections:
- net D13/SCK is gone; now on net D13: R1.1
- net D2: no longer J1.1 (Pin_1)
- net D3: no longer SW2.1
- net D4: no longer SW2.2
- net D5: now also SW2.1
- net D6: now also SW2.2
- net GND: now also J1.1 (Pin_1)
Other:
- note added: "D5 Backlight Enable"
- note added: "D6 Aux Light Enable"
- note removed: "D3 Backlight Enable"
- note removed: "D4 Aux Light Enable"

Commit message: Generated Final Rev 1 files for Hub and Slave
Parts:
- removed R10, R9: 1.8K, Resistor_SMD:R_0805_2012Metric, symbol Device:R
- J10, J11: now left out of the parts list
Connections:
- net GND: now also SW3.1
- net RESET: now also SW3.4 (A)
- net RXD: now also RJ1.2
- net TXD: now also RJ1.1
Changed lines of the file:
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@@
   (junction (at 207.01 21.59) (diameter 0) (color 0 0 0 0)
   )
+  (junction (at 38.1 35.56) (diameter 0) (color 0 0 0 0)
+  )
+  (junction (at 149.86 21.59) (diameter 0) (color 0 0 0 0)
+  )
   (junction (at 43.18 152.4) (diameter 0) (color 0 0 0 0)
   )
@@
   (junction (at 81.28 35.56) (diameter 0) (color 0 0 0 0)
   )
+  (junction (at 27.94 35.56) (diameter 0) (color 0 0 0 0)
+  )
   (junction (at 30.48 154.94) (diameter 0) (color 0 0 0 0)
   )
@@
     (stroke (width 0) (type default) (color 0 0 0 0))
   )
+  (wire (pts (xy 149.86 21.59) (xy 151.13 21.59))
+    (stroke (width 0) (type default) (color 0 0 0 0))
+  )
   (wire (pts (xy 252.73 25.4) (xy 255.27 25.4))
     (stroke (width 0) (type default) (color 0 0 0 0))
@@
     (stroke (width 0) (type default) (color 0 0 0 0))
   )
-  (wire (pts (xy 254 20.32) (xy 255.27 20.32))
+  (wire (pts (xy 252.73 20.32) (xy 255.27 20.32))
+    (stroke (width 0) (type default) (color 0 0 0 0))
+  )
+  (wire (pts (xy 38.1 33.02) (xy 38.1 35.56))
     (stroke (width 0) (type default) (color 0 0 0 0))
   )
@@
     (stroke (width 0) (type default) (color 0 0 0 0))
   )
-  (wire (pts (xy 148.59 21.59) (xy 151.13 21.59))
+  (wire (pts (xy 148.59 21.59) (xy 149.86 21.59))
     (stroke (width 0) (type default) (color 0 0 0 0))
   )
@@
     (stroke (width 0) (type default) (color 0 0 0 0))
   )
-  (wire (pts (xy 245.11 20.32) (xy 246.38 20.32))
-    (stroke (width 0) (type default) (color 0 0 0 0))
-  )
   (wire (pts (xy 83.82 147.32) (xy 86.36 147.32))
     (stroke (width 0) (type default) (color 0 0 0 0))
@@
     (stroke (width 0) (type default) (color 0 0 0 0))
   )
-  (wire (pts (xy 254 17.78) (xy 255.27 17.78))
+  (wire (pts (xy 27.94 33.02) (xy 27.94 35.56))
+    (stroke (width 0) (type default) (color 0 0 0 0))
+  )
+  (wire (pts (xy 252.73 17.78) (xy 255.27 17.78))
     (stroke (width 0) (type default) (color 0 0 0 0))
   )
@@
     (stroke (width 0) (type default) (color 0 0 0 0))
   )
-  (wire (pts (xy 245.11 17.78) (xy 246.38 17.78))
-    (stroke (width 0) (type default) (color 0 0 0 0))
-  )
   (wire (pts (xy 50.8 101.6) (xy 50.8 106.68))
     (stroke (width 0) (type default) (color 0 0 0 0))
@@
     )
   )
-  (global_label "RXD" (shape input) (at 245.11 17.78 180) (fields_autoplaced)
-    (effects (font (size 1.27 1.27)) (justify right))
-    (property "Intersheet References" "${INTERSHEET_REFS}" (id 0) (at 238.9474 17.7006 0)
-      (effects (font (size 1.27 1.27)) (justify right) hide)
-    )
-  )
   (global_label "D11" (shape bidirectional) (at 222.25 90.17 180) (fields_autoplaced)
     (effects (font (size 1.27 1.27)) (justify right))
@@
     )
   )
-  (global_label "TXD" (shape input) (at 245.11 20.32 180) (fields_autoplaced)
+  (global_label "TXD" (shape input) (at 252.73 17.78 180) (fields_autoplaced)
     (effects (font (size 1.27 1.27)) (justify right))
-    (property "Intersheet References" "${INTERSHEET_REFS}" (id 0) (at 239.2498 20.2406 0)
+    (property "Intersheet References" "${INTERSHEET_REFS}" (id 0) (at 246.8698 17.7006 0)
       (effects (font (size 1.27 1.27)) (justify right) hide)
     )
@@
     )
   )
+  (global_label "RXD" (shape input) (at 252.73 20.32 180) (fields_autoplaced)
+    (effects (font (size 1.27 1.27)) (justify right))
+    (property "Intersheet References" "${INTERSHEET_REFS}" (id 0) (at 246.5674 20.2406 0)
+      (effects (font (size 1.27 1.27)) (justify right) hide)
+    )
+  )
   (symbol (lib_id "Connector:Screw_Terminal_01x02") (at 271.78 114.3 0) (unit 1)
     (in_bom yes) (on_board yes) (fields_autoplaced)
@@
   )
   (symbol (lib_id "Connector:AVR-ISP-6") (at 87.63 74.93 0) (unit 1)
-    (in_bom yes) (on_board yes) (fields_autoplaced)
+    (in_bom no) (on_board yes) (fields_autoplaced)
     (property "Reference" "J10" (id 0) (at 78.74 72.3899 0)
       (effects (font (size 1.27 1.27)) (justify right))
@@
   )
   (symbol (lib_id "Connector:Conn_01x06_Female") (at 81.28 110.49 0) (mirror y) (unit 1)
-    (in_bom yes) (on_board yes)
+    (in_bom no) (on_board yes)
     (property "Reference" "J11" (id 0) (at 78.74 111.76 0))
     (property "Value" "Conn_01x06_Female" (id 1) (at 80.01 113.0299 0)
@@
     (pin "2")
   )
-  (symbol (lib_id "Device:R") (at 250.19 17.78 270) (unit 1)
-    (in_bom yes) (on_board yes)
-    (property "Reference" "R9" (id 0) (at 247.65 17.78 90))
-    (property "Value" "1.8K" (id 1) (at 251.46 17.78 90))
-    (property "Footprint" "Resistor_SMD:R_0805_2012Metric" (id 2) (at 250.19 16.002 90)
-      (effects (font (size 1.27 1.27)) hide)
-    )
-    (property "Datasheet" "~" (id 3) (at 250.19 17.78 0)
-      (effects (font (size 1.27 1.27)) hide)
-    )
-    (property "LCSC" "C17398" (id 4) (at 250.19 17.78 0)
-      (effects (font (size 1.27 1.27)) hide)
-    )
-    (pin "1")
-    (pin "2")
-  )
   (symbol (lib_id "Device:R") (at 48.26 29.21 0) (unit 1)
     (in_bom no) (on_board no) (fields_autoplaced)
@@
     (pin "1")
   )
-  (symbol (lib_id "Device:R") (at 250.19 20.32 270) (unit 1)
-    (in_bom yes) (on_board yes)
-    (property "Reference" "R10" (id 0) (at 247.65 20.32 90))
-    (property "Value" "1.8K" (id 1) (at 251.46 20.32 90))
-    (property "Footprint" "Resistor_SMD:R_0805_2012Metric" (id 2) (at 250.19 18.542 90)
-      (effects (font (size 1.27 1.27)) hide)
-    )
-    (property "Datasheet" "~" (id 3) (at 250.19 20.32 0)
-      (effects (font (size 1.27 1.27)) hide)
-    )
-    (property "LCSC" "C17398" (id 4) (at 250.19 20.32 0)
-      (effects (font (size 1.27 1.27)) hide)
-    )
-    (pin "1")
-    (pin "2")
-  )
   (symbol (lib_id "Device:C") (at 105.41 31.75 0) (unit 1)
     (in_bom yes) (on_board yes) (fields_autoplaced)
@@
     (pin "2")
   )
+  (symbol (lib_id "power:PWR_FLAG") (at 149.86 21.59 0) (unit 1)
+    (in_bom yes) (on_board yes)
+    (property "Reference" "#FLG0101" (id 0) (at 149.86 19.685 0)
+      (effects (font (size 1.27 1.27)) hide)
+    )
+    (property "Value" "PWR_FLAG" (id 1) (at 156.21 19.05 0))
+    (property "Footprint" "" (id 2) (at 149.86 21.59 0)
+      (effects (font (size 1.27 1.27)) hide)
+    )
+    (property "Datasheet" "~" (id 3) (at 149.86 21.59 0)
+      (effects (font (size 1.27 1.27)) hide)
+    )
+    (pin "1")
+  )
   (symbol (lib_id "power:GND") (at 38.1 93.98 180) (unit 1)
     (in_bom yes) (on_board yes) (fields_autoplaced)
@@
   )
   (symbol_instances
+    (path "/e3deca73-d735-4dce-bffc-182df1d4683e"
+      (reference "#FLG0101") (unit 1) (value "PWR_FLAG") (footprint "")
+    )
     (path "/d0589162-1c09-49d5-9b0b-72174a6be181"
       (reference "#PWR0101") (unit 1) (value "+5V") (footprint "")
@@
       (reference "R8") (unit 1) (value "1.8K") (footprint "Resistor_SMD:R_0805_2012Metric")
     )
-    (path "/739faa62-306a-4993-b412-ba4895b74608"
-      (reference "R9") (unit 1) (value "1.8K") (footprint "Resistor_SMD:R_0805_2012Metric")
-    )
-    (path "/897a3989-0eff-4e30-863b-c9bc5cde57f3"
-      (reference "R10") (unit 1) (value "1.8K") (footprint "Resistor_SMD:R_0805_2012Metric")
-    )
     (path "/b0d080a8-fb27-4ca9-906d-778ef01ddc29"
