File: KiCad PCBs/External Connectors/External Connectors.kicad_sch (KiCad schematic)
At the start: 8 parts, among them J1 Conn_02x04_Top_Bottom, J2 Conn_02x04_Top_Bottom, J3 USB_B, J4 USB_A

Commit message: Updated External Connectors BOM
Parts:
- J1, J2: now in the parts list
Changed lines of the file:
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@@
   )
   (symbol (lib_id "Connector_Generic:Conn_02x04_Top_Bottom") (at 130.81 83.82 0) (unit 1)
-    (in_bom no) (on_board yes)
+    (in_bom yes) (on_board yes)
     (property "Reference" "J1" (id 0) (at 132.08 77.47 0))
     (property "Value" "Conn_02x04_Top_Bottom" (id 1) (at 132.08 77.47 0)
@@
   )
   (symbol (lib_id "Connector_Generic:Conn_02x04_Top_Bottom") (at 130.81 102.87 0) (unit 1)
-    (in_bom no) (on_board yes)
+    (in_bom yes) (on_board yes)
     (property "Reference" "J2" (id 0) (at 132.08 96.52 0))
     (property "Value" "Conn_02x04_Top_Bottom" (id 1) (at 132.08 96.52 0)
