File: KiCad PCBs/Mega Slave/Mega Slave.kicad_sch (KiCad schematic)
At the start: 76 parts, among them J1 AVR-ISP-6, J10 Screw_Terminal_01x02, J11 Screw_Terminal_01x02, J12 Screw_Terminal_01x02, J13 Screw_Terminal_01x02, J14 Screw_Terminal_01x02, J15 Screw_Terminal_01x02, J16 Screw_Terminal_01x02, J17 Screw_Terminal_01x02, J18 Screw_Terminal_01x02, J19 Screw_Terminal_01x02, J2 Screw_Terminal_01x02, J20 Screw_Terminal_01x02, J21 Screw_Terminal_01x02, J22 Screw_Terminal_01x02, J23 Screw_Terminal_01x02, J24 Screw_Terminal_01x02, J25 Screw_Terminal_01x02, J26 Screw_Terminal_01x02, J27 Screw_Terminal_01x02, J28 Screw_Terminal_01x02, J29 Screw_Terminal_01x02, J3 Screw_Terminal_01x02, J30 Screw_Terminal_01x02, J31 Screw_Terminal_01x02, J32 Screw_Terminal_01x02, J33 Screw_Terminal_01x02, J34 Screw_Terminal_01x02, J35 Screw_Terminal_01x02, J36 Screw_Terminal_01x02, J37 Screw_Terminal_01x02, J38 Screw_Terminal_01x02, J4 Screw_Terminal_01x02, J5 Screw_Terminal_01x02, J6 Screw_Terminal_01x02, J7 Screw_Terminal_01x02, J8 Screw_Terminal_01x02, J9 Screw_Terminal_01x02, SW1 SW_MEC_5E, SW2 SW_DIP_x02, SW3 SW_DIP_x02, U1 ATmega2560-16A, U2 MAX487ESA+T, U3 AMS1117-5.0, U4 ULN2003A, Y1 Crystal_GND24

Commit message: Mega Slave WIP
Parts:
- H1, H2, H3, H4: renamed from H?; now left out of the parts list
- J10, J11, J12, J13, J14, J15, J16, J17, J18, J19, J2, J20, J21, J22, J23, J24, J25, J26, J27, J28, J29, J3, J30, J31, J32, J33, J34, J35, J36, J37, J38, J4, J5, J6, J7, J8, J9: footprint A10 KiCad Libraries:CONN-TH_WJ126V-5.0-2P -> A10 KiCad Libraries:CONN-TH_XY308-2.54-2P; LCSC C8404 -> C557685
- J40, J41: renamed from J?; footprint A10 KiCad Libraries:CONN-TH_WJ126V-5.0-2P -> A10 KiCad Libraries:CONN-TH_XY308-2.54-2P; LCSC C8404 -> C557685
- gave numbers to parts that had none: 5
- renumbered C1 to C14
Connections:
- net D42: now also U1.42 (PL7/D42)
- net D43: now also U1.41 (PL6/D43)
- net D48: now also U1.36 (PL1/D48)
- net D49: now also U1.35 (PL0/D49)
- net D50: now also J1.1 (MISO)
- net D51: now also J1.4 (MOSI)
- net D52: now also J1.3 (SCK)
- no-connect marks 23 -> 19
Other:
- moved on the sheet: C13, J28, J29, J30, J31, J32, J33, J34, J35, J36, J37, J38

Commit message: Mega Slave Initial Routing
Connections:
- net D16: now also U1.13 (PH1/TXD2/D16)
- net D18: no longer U1.13 (PH1/TXD2/D18)
