File: KiCad PCBs/Nano Shield/Nano Shield.kicad_sch (KiCad schematic)
At the start: 34 parts, among them J1 Conn_01x15_Female, J10 Screw_Terminal_01x02, J11 Screw_Terminal_01x02, J12 Screw_Terminal_01x02, J13 Screw_Terminal_01x02, J14 Screw_Terminal_01x02, J15 Screw_Terminal_01x02, J16 Screw_Terminal_01x02, J17 Screw_Terminal_01x02, J18 Screw_Terminal_01x02, J2 Conn_01x15_Female, J3 Screw_Terminal_01x02, J4 Screw_Terminal_01x02, J5 Screw_Terminal_01x02, J6 Screw_Terminal_01x02, J7 Screw_Terminal_01x02, J8 Screw_Terminal_01x02, J9 Screw_Terminal_01x02, SW1 SW_DIP_x02, SW2 SW_DIP_x02, U1 MAX487ESA+T, U2 AMS1117-5.0, U3 ULN2003A

Commit message: Finished Nano Shield
Parts:
- H1: footprint (none) -> MountingHole:MountingHole_3.2mm_M3
- J10, J11, J12, J13, J14, J15, J16, J17, J18, J3, J4, J5, J6, J7, J8, J9: footprint A10 KiCad Libraries:CONN-TH_XY308-2.54-2P -> A10 KiCad Libraries:CONN-TH_WJ126V-5.0-2P
Connections:
- net +12V: now also J17.2 (Pin_2), J18.2 (Pin_2); no longer J17.1 (Pin_1), J18.1 (Pin_1)
- net +3V3: now also J16.2 (Pin_2); no longer J16.1 (Pin_1)
- net A0/D14: now also J8.2 (Pin_2); no longer J8.1 (Pin_1)
- net A1/D15: now also J9.1 (Pin_1); no longer J9.2 (Pin_2)
- net A2/D16: now also J9.2 (Pin_2); no longer J9.1 (Pin_1)
- net A3/D17: now also J10.1 (Pin_1); no longer J10.2 (Pin_2)
- net A4/D18: now also J10.2 (Pin_2); no longer J10.1 (Pin_1)
- net A5/D19: now also J11.1 (Pin_1); no longer J11.2 (Pin_2)
- net A6: now also J11.2 (Pin_2); no longer J11.1 (Pin_1)
- net A7: now also J12.1 (Pin_1); no longer J12.2 (Pin_2)
- net AUX_BASE: now also SW2.1; no longer SW2.3
- net AUX_GND: now also J18.1 (Pin_1); no longer J18.2 (Pin_2)
- net BACKLIGHT_BASE: now also SW2.2; no longer SW2.4
- net BACKLIGHT_GND: now also J17.1 (Pin_1); no longer J17.2 (Pin_2)
- net D10~/SS: now also J6.2 (Pin_2); no longer J6.1 (Pin_1)
- net D11~/MOSI: now also J7.1 (Pin_1); no longer J7.2 (Pin_2)
- net D12/MISO: now also J7.2 (Pin_2); no longer J7.1 (Pin_1)
- net D13/SCK: now also J8.1 (Pin_1); no longer J8.2 (Pin_2)
- net D3~: now also J3.1 (Pin_1); no longer J3.2 (Pin_2)
- net D4: now also J3.2 (Pin_2); no longer J3.1 (Pin_1)
- net D5~/BACKLIGHT: now also J4.1 (Pin_1), SW2.3; no longer J4.2 (Pin_2), SW2.1
- net D6~/AUX_LIGHT: now also J4.2 (Pin_2), SW2.4; no longer J4.1 (Pin_1), SW2.2
- net D7: now also J5.1 (Pin_1); no longer J5.2 (Pin_2)
- net D8: now also J5.2 (Pin_2); no longer J5.1 (Pin_1)
- net D9~: now also J6.1 (Pin_1); no longer J6.2 (Pin_2)
- net GND: now also J12.2 (Pin_2), J16.1 (Pin_1), SW1.4; no longer J12.1 (Pin_1), J16.2 (Pin_2), SW1.1
- net RS485-: now also SW1.3; no longer SW1.2
- net RS485_GND: now also SW1.1; no longer SW1.4
- net at R3.2: now also SW1.2; no longer SW1.3
