File: PCBs/Panels/UFC/UFC.kicad_sch (KiCad schematic)
At the start: 94 parts, among them J1 Conn_02x11_Top_Bottom, J2 Conn_02x11_Top_Bottom, SW1 1, SW10 STEER +, SW11 DEPR +, SW12 4, SW13 5, SW14 6, SW15 0, SW16 LTR, SW17 MK, SW18 COM 1, SW19 COM SEC, SW2 2, SW20 IFF, SW21 DATA -, SW22 SEL -, SW23 STEER -, SW24 DEPR -, SW25 7, SW26 8, SW27 9, SW28 SPC, SW29 CLR, SW3 3, SW30 ALT ALRT, SW31 COM 2, SW32 ECCM, SW33 IDM R/T, SW34 INTEN <, SW35 INTEN >, SW4 HACK, SW5 FUNC, SW6 ENT, SW7 MASTER CAUTION, SW8 DATA +, SW9 SEL +

Commit message: UFC Completed
Parts:
- gave numbers to parts that had none: 1
Connections:
- net GND: now also SW10.2, SW11.2, SW12.2, SW13.2, SW14.2, SW15.2, SW16.2, SW17.2, SW18.2, SW19.2, SW20.2, SW21.2, SW22.2, SW23.2, SW24.2, SW25.2, SW26.2, SW27.2, SW28.2, SW29.2, SW30.2, SW31.2, SW32.2, SW33.2, SW34.2, SW35.2, SW4.2, SW5.2, SW6.2, SW7.2, SW8.2, SW9.2
