File: PCBs/Slaves/Mega Slave/Mega Slave.kicad_pcb (KiCad board)
At the start: 2 copper layers, 157 x 80 mm, 76 parts, among them J1 AVR-ISP-6, J10 Screw_Terminal_01x02, J11 Screw_Terminal_01x02, J12 Screw_Terminal_01x02, J13 Screw_Terminal_01x02, J14 Screw_Terminal_01x02, J15 Screw_Terminal_01x02, J16 Screw_Terminal_01x02, J17 Screw_Terminal_01x02, J18 Screw_Terminal_01x02, J19 Screw_Terminal_01x02, J2 Screw_Terminal_01x02, J20 Screw_Terminal_01x02, J21 Screw_Terminal_01x02, J22 Screw_Terminal_01x02, J23 Screw_Terminal_01x02, J24 Screw_Terminal_01x02, J25 Screw_Terminal_01x02, J26 Screw_Terminal_01x02, J27 Screw_Terminal_01x02, J28 Screw_Terminal_01x02, J29 Screw_Terminal_01x02, J3 Screw_Terminal_01x02, J30 Screw_Terminal_01x02, J31 Screw_Terminal_01x02, J32 Screw_Terminal_01x02, J33 Screw_Terminal_01x02, J34 Screw_Terminal_01x02, J35 Screw_Terminal_01x02, J36 Screw_Terminal_01x02, J37 Screw_Terminal_01x02, J39 Conn_01x06_Female, J4 Screw_Terminal_01x02, J40 Screw_Terminal_01x02, J41 Screw_Terminal_01x02, J5 Screw_Terminal_01x02, J6 Screw_Terminal_01x02, J7 Screw_Terminal_01x02, J8 Screw_Terminal_01x02, J9 Screw_Terminal_01x02, SW1 SW_MEC_5E, SW2 SW_DIP_x02, SW3 SW_DIP_x02, U1 ATmega2560-16A, U2 MAX487ESA+T, U3 AMS1117-5.0, U4 ULN2003A, U5 MAX487ESA+T, Y1 Crystal_GND24

Commit message: Mega Slave Rev. 2 Completed
Parts:
- added D3: LED, LED_SMD:LED_0603_1608Metric, F.Cu at (225.5, 114.0)
- added R7: 1K, Resistor_SMD:R_0805_2012Metric, F.Cu at (223.5, 114.0)
- added REF**: OSHW-Logo2_14.6x12mm_Copper, Symbol:OSHW-Logo2_14.6x12mm_Copper, F.Cu at (101.0, 108.5)
- moved R3 4.27 mm to (197.5, 125.5), turned to 180 degrees
- moved D1 2.46 mm to (197.5, 127.5), turned to 180 degrees
Routing:
- net GND: track 0.00 -> 18.4 mm, vias 0 -> 72
- net D3: track 80.0 -> 87.9 mm, vias 0 -> 2
- net D13: track 155.2 -> 162.6 mm, vias 4 -> 6
- net Net-(D3-Pad2): track 0.00 -> 2.05 mm
- net BACKLIGHT_GND: track 24.5 -> 22.9 mm
- net D46: track 95.8 -> 94.8 mm
- net D24: track 81.1 -> 80.6 mm

Commit message: Completed Caution Panel
Other:
- board text added: "150MM →"
- board text added: "BRRRRRRRRT"
- board text added: "M3"
- board text added: "← 73MM"
Changed lines of the file:
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@@
     )
   )
+  (gr_circle (center 161.02 101.974915) (end 191.02 101.974915) (layer "B.SilkS") (width 0.127) (fill none))
   (gr_arc (start 85.045117 141.479999) (mid 82.561086 140.470825) (end 81.52 138) (layer "Edge.Cuts") (width 0.1016))
   (gr_line (start 85.045117 141.479999) (end 235 141.474915) (layer "Edge.Cuts") (width 0.1016))
@@
   (gr_arc (start 238.525117 137.949798) (mid 237.486741 140.436539) (end 235 141.474915) (layer "Edge.Cuts") (width 0.1016))
   (gr_arc (start 81.520001 65) (mid 82.529175 62.51597) (end 85 61.474883) (layer "Edge.Cuts") (width 0.1016))
+  (gr_text "BRRRRRRRRT" (at 162.02 101.974915 15) (layer "B.SilkS")
+    (effects (font (size 7.62 7.62) (thickness 0.8128)) (justify mirror))
+  )
+  (gr_text "← 73MM" (at 232.52 126.974915 90) (layer "B.SilkS")
+    (effects (font (size 1.2192 1.2192) (thickness 0.1524)) (justify mirror))
+  )
+  (gr_text "M3" (at 235.02 134.974915) (layer "B.SilkS")
+    (effects (font (size 1.2192 1.2192) (thickness 0.1524)) (justify mirror))
+  )
+  (gr_text "150MM →" (at 225.02 135.974915) (layer "B.SilkS")
+    (effects (font (size 1.2192 1.2192) (thickness 0.1524)) (justify mirror))
+  )
   (gr_text "WarthogAtHome.com" (at 168.315086 126.474915) (layer "F.SilkS")
     (effects (font (size 1.3208 1.3208) (thickness 0.2032)) (justify right))
