File: PCBs/Slaves/Mega Slave/Mega Slave.kicad_sch (KiCad schematic)
At the start: 76 parts, among them J1 AVR-ISP-6, J10 Screw_Terminal_01x02, J11 Screw_Terminal_01x02, J12 Screw_Terminal_01x02, J13 Screw_Terminal_01x02, J14 Screw_Terminal_01x02, J15 Screw_Terminal_01x02, J16 Screw_Terminal_01x02, J17 Screw_Terminal_01x02, J18 Screw_Terminal_01x02, J19 Screw_Terminal_01x02, J2 Screw_Terminal_01x02, J20 Screw_Terminal_01x02, J21 Screw_Terminal_01x02, J22 Screw_Terminal_01x02, J23 Screw_Terminal_01x02, J24 Screw_Terminal_01x02, J25 Screw_Terminal_01x02, J26 Screw_Terminal_01x02, J27 Screw_Terminal_01x02, J28 Screw_Terminal_01x02, J29 Screw_Terminal_01x02, J3 Screw_Terminal_01x02, J30 Screw_Terminal_01x02, J31 Screw_Terminal_01x02, J32 Screw_Terminal_01x02, J33 Screw_Terminal_01x02, J34 Screw_Terminal_01x02, J35 Screw_Terminal_01x02, J36 Screw_Terminal_01x02, J37 Screw_Terminal_01x02, J38 Screw_Terminal_01x02, J39 Conn_01x06_Female, J4 Screw_Terminal_01x02, J40 Screw_Terminal_01x02, J41 Screw_Terminal_01x02, J5 Screw_Terminal_01x02, J6 Screw_Terminal_01x02, J7 Screw_Terminal_01x02, J8 Screw_Terminal_01x02, J9 Screw_Terminal_01x02, SW1 SW_MEC_5E, SW2 SW_DIP_x02, SW3 SW_DIP_x02, U1 ATmega2560-16A, U2 MAX487ESA+T, U3 AMS1117-5.0, U4 ULN2003A, Y1 Crystal_GND24

Commit message: Rearranged files
Parts:
- removed J38: Screw_Terminal_01x02, A10 KiCad Libraries:CONN-TH_XY308-2.54-2P, symbol Connector:Screw_Terminal_01x02
- added U5: MAX487ESA+T, Package_DIP:DIP-8_W7.62mm, symbol A10:MAX487
- J10, J11, J12, J13, J14, J15, J16, J17, J18, J19, J2, J20, J21, J22, J23, J24, J25, J26, J27, J28, J29, J3, J30, J31, J32, J33, J34, J35, J36, J37, J4, J40, J41, J5, J6, J7, J8, J9: footprint A10 KiCad Libraries:CONN-TH_XY308-2.54-2P -> A10 KiCad Libraries:CONN-TH_WJ126V-5.0-2P
Connections:
- net +12V: no longer J36.2 (Pin_2)
- net +5V: now also U5.8 (VCC); no longer J37.2 (Pin_2)
- net A0: now also J28.2 (Pin_2); no longer J28.1 (Pin_1)
- net A1: now also J28.1 (Pin_1); no longer J28.2 (Pin_2)
- net A10: now also J33.2 (Pin_2); no longer J33.1 (Pin_1)
- net A11: now also J33.1 (Pin_1); no longer J33.2 (Pin_2)
- net A12: now also J34.2 (Pin_2); no longer J34.1 (Pin_1)
- net A13: now also J34.1 (Pin_1); no longer J34.2 (Pin_2)
- net A14: now also J35.2 (Pin_2); no longer J35.1 (Pin_1)
- net A15: now also J35.1 (Pin_1); no longer J35.2 (Pin_2)
- net A2: now also J29.2 (Pin_2); no longer J29.1 (Pin_1)
- net A3: now also J29.1 (Pin_1); no longer J29.2 (Pin_2)
- net A4: now also J30.2 (Pin_2); no longer J30.1 (Pin_1)
- net A5: now also J30.1 (Pin_1); no longer J30.2 (Pin_2)
- net A6: now also J31.2 (Pin_2); no longer J31.1 (Pin_1)
- net A7: now also J31.1 (Pin_1); no longer J31.2 (Pin_2)
- net A8: now also J32.2 (Pin_2); no longer J32.1 (Pin_1)
- net A9: now also J32.1 (Pin_1); no longer J32.2 (Pin_2)
- net D10: now also J5.1 (Pin_1); no longer J5.2 (Pin_2)
- net D11: now also J6.2 (Pin_2); no longer J6.1 (Pin_1)
- net D12: now also J6.1 (Pin_1); no longer J6.2 (Pin_2)
- net D13: now also J7.2 (Pin_2); no longer J7.1 (Pin_1)
- net D14: now also J7.1 (Pin_1); no longer J7.2 (Pin_2)
- net D15: now also J8.2 (Pin_2); no longer J8.1 (Pin_1)
- net D16: now also J8.1 (Pin_1); no longer J8.2 (Pin_2)
- net D17: now also J9.2 (Pin_2); no longer J9.1 (Pin_1)
- net D18: now also J9.1 (Pin_1); no longer J9.2 (Pin_2)
- net D19: now also J10.2 (Pin_2); no longer J10.1 (Pin_1)
- net D2: now also U5.2 (~{RE}), U5.3 (DE)
- net D20: now also J10.1 (Pin_1); no longer J10.2 (Pin_2)
- net D21: now also J11.2 (Pin_2); no longer J11.1 (Pin_1)
- net D22: now also J11.1 (Pin_1); no longer J11.2 (Pin_2)
- net D23: now also J12.2 (Pin_2); no longer J12.1 (Pin_1)
- net D24: now also J12.1 (Pin_1); no longer J12.2 (Pin_2)
- net D25: now also J13.2 (Pin_2); no longer J13.1 (Pin_1)
- net D26: now also J13.1 (Pin_1); no longer J13.2 (Pin_2)
- net D27: now also J14.2 (Pin_2); no longer J14.1 (Pin_1)
- net D28: now also J14.1 (Pin_1); no longer J14.2 (Pin_2)
- net D29: now also J15.2 (Pin_2); no longer J15.1 (Pin_1)
- net D3: now also J2.2 (Pin_2); no longer J2.1 (Pin_1)
- net D30: now also J15.1 (Pin_1); no longer J15.2 (Pin_2)
- net D31: now also J16.2 (Pin_2); no longer J16.1 (Pin_1)
- net D32: now also J16.1 (Pin_1); no longer J16.2 (Pin_2)
- net D33: now also J17.2 (Pin_2); no longer J17.1 (Pin_1)
- net D34: now also J17.1 (Pin_1); no longer J17.2 (Pin_2)
- net D35: now also J18.2 (Pin_2); no longer J18.1 (Pin_1)
- net D36: now also J18.1 (Pin_1); no longer J18.2 (Pin_2)
- net D37: now also J19.2 (Pin_2); no longer J19.1 (Pin_1)
- net D38: now also J19.1 (Pin_1); no longer J19.2 (Pin_2)
- net D39: now also J20.2 (Pin_2); no longer J20.1 (Pin_1)
- net D4: now also J2.1 (Pin_1); no longer J2.2 (Pin_2)
- net D40: now also J20.1 (Pin_1); no longer J20.2 (Pin_2)
- net D41: now also J21.2 (Pin_2); no longer J21.1 (Pin_1)
- net D42: now also J21.1 (Pin_1); no longer J21.2 (Pin_2)
- net D43: now also J22.2 (Pin_2); no longer J22.1 (Pin_1)
- net D44: now also J22.1 (Pin_1); no longer J22.2 (Pin_2)
- net D45: now also J23.2 (Pin_2); no longer J23.1 (Pin_1)
- net D46: now also J23.1 (Pin_1); no longer J23.2 (Pin_2)
- net D47: now also J24.2 (Pin_2); no longer J24.1 (Pin_1)
- net D48: now also J24.1 (Pin_1); no longer J24.2 (Pin_2)
- net D49: now also J25.2 (Pin_2); no longer J25.1 (Pin_1)
- net D5: now also J3.2 (Pin_2); no longer J3.1 (Pin_1)
- net D50: now also J25.1 (Pin_1); no longer J25.2 (Pin_2)
- net D51: now also J26.2 (Pin_2); no longer J26.1 (Pin_1)
- net D52: now also J26.1 (Pin_1); no longer J26.2 (Pin_2)
- net D53: now also J27.2 (Pin_2); no longer J27.1 (Pin_1)
- net D6: now also J3.1 (Pin_1); no longer J3.2 (Pin_2)
- net D7: now also J4.2 (Pin_2); no longer J4.1 (Pin_1)
- net D8: now also J4.1 (Pin_1); no longer J4.2 (Pin_2)
- net D9: now also J5.2 (Pin_2); no longer J5.1 (Pin_1)
- net GND: now also J27.1 (Pin_1), J36.2 (Pin_2), J37.2 (Pin_2); no longer J27.2 (Pin_2)
- net RS485+: now also U5.6 (A)
- net RS485-: now also U5.7 (B)
- net RS485_GND: now also U5.5 (GND)
- net RXD: now also U5.1 (RO)
- net TXD: now also U5.4 (DI)

Commit message: Mega Slave Rev. 2 Completed
Parts:
- added D3: LED, LED_SMD:LED_0603_1608Metric, symbol Device:LED
- added R7: 1K, Resistor_SMD:R_0805_2012Metric, symbol Device:R
Connections:
- net D3: now also R7.1
- net GND: now also D3.1 (K)
- new net: D3.2 (A), R7.2
Other:
- note added: "D3"
- note added: "Extra LEDs"
Changed lines of the file:
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@@
     (stroke (width 0) (type default) (color 0 0 0 0))
   )
+  (wire (pts (xy 90.17 97.79) (xy 92.71 97.79))
+    (stroke (width 0) (type default) (color 0 0 0 0))
+  )
   (wire (pts (xy 35.56 113.03) (xy 35.56 115.57))
     (stroke (width 0) (type default) (color 0 0 0 0))
@@
     (stroke (width 0) (type default) (color 0 0 0 0))
   )
+  (wire (pts (xy 80.01 97.79) (xy 82.55 97.79))
+    (stroke (width 0) (type default) (color 0 0 0 0))
+  )
   (wire (pts (xy 115.57 26.67) (xy 127 26.67))
     (stroke (width 0) (type default) (color 0 0 0 0))
@@
     (stroke (width 0) (type default) (color 0 0 0 0))
   )
+  (polyline (pts (xy 110.49 105.41) (xy 63.5 105.41))
+    (stroke (width 0) (type default) (color 0 0 0 0))
+  )
   (wire (pts (xy 95.25 16.51) (xy 95.25 19.05))
     (stroke (width 0) (type default) (color 0 0 0 0))
@@
     (stroke (width 0) (type default) (color 0 0 0 0))
   )
+  (wire (pts (xy 100.33 97.79) (xy 102.87 97.79))
+    (stroke (width 0) (type default) (color 0 0 0 0))
+  )
   (polyline (pts (xy 12.7 119.38) (xy 63.5 119.38))
     (stroke (width 0) (type default) (color 0 0 0 0))
@@
     (stroke (width 0) (type default) (color 0 0 0 0))
   )
+  (polyline (pts (xy 110.49 87.63) (xy 110.49 105.41))
+    (stroke (width 0) (type default) (color 0 0 0 0))
+  )
   (wire (pts (xy 92.71 26.67) (xy 95.25 26.67))
     (stroke (width 0) (type default) (color 0 0 0 0))
@@
     (effects (font (size 1.27 1.27)) (justify left bottom))
   )
+  (text "D3" (at 66.04 99.06 0)
+    (effects (font (size 1.27 1.27)) (justify left bottom))
+  )
   (text "Right Green\nLED" (at 274.32 43.18 0)
     (effects (font (size 1.016 1.016)) (justify left bottom))
@@
     (effects (font (size 0.381 0.381)) (justify left bottom))
   )
+  (text "Extra LEDs" (at 66.04 91.44 0)
+    (effects (font (size 1.27 1.27)) (justify left bottom))
+  )
   (text "D4 Backlight Enable" (at 198.755 33.02 0)
     (effects (font (size 0.381 0.381)) (justify left bottom))
@@
     )
   )
+  (global_label "D3" (shape input) (at 80.01 97.79 180) (fields_autoplaced)
+    (effects (font (size 1.27 1.27)) (justify right))
+    (property "Intersheet References" "${INTERSHEET_REFS}" (id 0) (at 75.1174 97.7106 0)
+      (effects (font (size 1.27 1.27)) (justify right) hide)
+    )
+  )
   (global_label "RESET" (shape input) (at 124.46 48.26 180) (fields_autoplaced)
     (effects (font (size 1.27 1.27)) (justify right))
@@
     (pin "8")
   )
+  (symbol (lib_id "Device:R") (at 86.36 97.79 90) (unit 1)
+    (in_bom yes) (on_board yes) (fields_autoplaced)
+    (property "Reference" "R7" (id 0) (at 86.36 91.44 90))
+    (property "Value" "1K" (id 1) (at 86.36 93.98 90))
+    (property "Footprint" "Resistor_SMD:R_0805_2012Metric" (id 2) (at 86.36 99.568 90)
+      (effects (font (size 1.27 1.27)) hide)
+    )
+    (property "Datasheet" "~" (id 3) (at 86.36 97.79 0)
+      (effects (font (size 1.27 1.27)) hide)
+    )
+    (property "LCSC" "C17513" (id 4) (at 86.36 97.79 0)
+      (effects (font (size 1.27 1.27)) hide)
+    )
+    (pin "1")
+    (pin "2")
+  )
   (symbol (lib_id "power:+5V") (at 38.1 46.99 270) (unit 1)
     (in_bom yes) (on_board yes) (fields_autoplaced)
@@
     (pin "2")
   )
+  (symbol (lib_id "power:GND") (at 102.87 97.79 90) (unit 1)
+    (in_bom yes) (on_board yes)
+    (property "Reference" "#PWR?" (id 0) (at 109.22 97.79 0)
+      (effects (font (size 1.27 1.27)) hide)
+    )
+    (property "Value" "GND" (id 1) (at 107.95 97.79 0))
+    (property "Footprint" "" (id 2) (at 102.87 97.79 0)
+      (effects (font (size 1.27 1.27)) hide)
+    )
+    (property "Datasheet" "" (id 3) (at 102.87 97.79 0)
+      (effects (font (size 1.27 1.27)) hide)
+    )
+    (pin "1")
+  )
   (symbol (lib_id "Switch:SW_MEC_5E") (at 35.56 25.4 0) (unit 1)
     (in_bom yes) (on_board yes) (fields_autoplaced)
@@
     (pin "2")
   )
+  (symbol (lib_id "Device:LED") (at 96.52 97.79 180) (unit 1)
+    (in_bom yes) (on_board yes)
+    (property "Reference" "D3" (id 0) (at 97.79 91.44 0))
+    (property "Value" "LED" (id 1) (at 97.79 93.98 0))
+    (property "Footprint" "LED_SMD:LED_0603_1608Metric" (id 2) (at 96.52 97.79 0)
+      (effects (font (size 1.27 1.27)) hide)
+    )
+    (property "Datasheet" "~" (id 3) (at 96.52 97.79 0)
+      (effects (font (size 1.27 1.27)) hide)
+    )
+    (property "LCSC" "C72041" (id 4) (at 96.52 97.79 0)
+      (effects (font (size 1.27 1.27)) hide)
+    )
+    (pin "1")
+    (pin "2")
+  )
   (symbol (lib_id "A10:MAX487") (at 35.56 99.06 0) (unit 1)
     (in_bom yes) (on_board yes)
@@
       (reference "#PWR0102") (unit 1) (value "GND") (footprint "")
     )
+    (path "/6c80d467-0e88-4ab5-b1d4-c89cf316000b"
+      (reference "#PWR?") (unit 1) (value "GND") (footprint "")
+    )
     (path "/72389c6e-73d3-4ab2-b7b7-a5c7261c1812"
       (reference "C1") (unit 1) (value "4.7uF") (footprint "A10 KiCad Libraries:C0805")
@@
       (reference "D2") (unit 1) (value "LED") (footprint "LED_SMD:LED_0603_1608Metric")
     )
+    (path "/929bef45-85fe-4757-9024-14a5d5385036"
+      (reference "D3") (unit 1) (value "LED") (footprint "LED_SMD:LED_0603_1608Metric")
+    )
     (path "/f8745f10-1505-43ab-a00d-5db2752af72e"
       (reference "H1") (unit 1) (value "MountingHole") (footprint "MountingHole:MountingHole_3.2mm_M3")
@@
       (reference "R6") (unit 1) (value "1K") (footprint "Resistor_SMD:R_0805_2012Metric")
     )
+    (path "/67476c28-106b-4010-b856-1e4c3cc5b479"
+      (reference "R7") (unit 1) (value "1K") (footprint "Resistor_SMD:R_0805_2012Metric")
+    )
     (path "/a86cf0e6-4d11-4fc0-b643-cc37acff4da7"

Commit message: Fixed part number of screw terminals
Parts:
- J10, J11, J12, J13, J14, J15, J16, J17, J18, J19, J2, J20, J21, J22, J23, J24, J25, J26, J27, J28, J29, J3, J30, J31, J32, J33, J34, J35, J36, J37, J4, J40, J41, J5, J6, J7, J8, J9: LCSC C557685 -> C8404
Changed lines of the file:
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@@
       (effects (font (size 1.27 1.27)) hide)
     )
-    (property "LCSC" "C557685" (id 4) (at 271.78 109.22 0)
+    (property "LCSC" "C8404" (id 4) (at 271.78 109.22 0)
       (effects (font (size 1.27 1.27)) hide)
     )
@@
       (effects (font (size 1.27 1.27)) hide)
     )
-    (property "LCSC" "C557685" (id 4) (at 227.33 144.78 0)
+    (property "LCSC" "C8404" (id 4) (at 227.33 144.78 0)
       (effects (font (size 1.27 1.27)) hide)
     )
@@
       (effects (font (size 1.27 1.27)) hide)
     )
-    (property "LCSC" "C557685" (id 4) (at 227.33 139.7 0)
+    (property "LCSC" "C8404" (id 4) (at 227.33 139.7 0)
       (effects (font (size 1.27 1.27)) hide)
     )
@@
       (effects (font (size 1.27 1.27)) hide)
     )
-    (property "LCSC" "C557685" (id 4) (at 204.47 121.92 0)
+    (property "LCSC" "C8404" (id 4) (at 204.47 121.92 0)
       (effects (font (size 1.27 1.27)) hide)
     )
@@
       (effects (font (size 1.27 1.27)) hide)
     )
-    (property "LCSC" "C557685" (id 4) (at 204.47 86.36 0)
+    (property "LCSC" "C8404" (id 4) (at 204.47 86.36 0)
       (effects (font (size 1.27 1.27)) hide)
     )
@@
       (effects (font (size 1.27 1.27)) hide)
     )
-    (property "LCSC" "C557685" (id 4) (at 204.47 63.5 0)
+    (property "LCSC" "C8404" (id 4) (at 204.47 63.5 0)
       (effects (font (size 1.27 1.27)) hide)
     )
@@
       (effects (font (size 1.27 1.27)) hide)
     )
-    (property "LCSC" "C557685" (id 4) (at 227.33 63.5 0)
+    (property "LCSC" "C8404" (id 4) (at 227.33 63.5 0)
       (effects (font (size 1.27 1.27)) hide)
     )
@@
       (effects (font (size 1.27 1.27)) hide)
     )
-    (property "LCSC" "C557685" (id 4) (at 204.47 58.42 0)
+    (property "LCSC" "C8404" (id 4) (at 204.47 58.42 0)
       (effects (font (size 1.27 1.27)) hide)
     )
@@
       (effects (font (size 1.27 1.27)) hide)
     )
-    (property "LCSC" "C557685" (id 4) (at 227.33 58.42 0)
+    (property "LCSC" "C8404" (id 4) (at 227.33 58.42 0)
       (effects (font (size 1.27 1.27)) hide)
     )
@@
       (effects (font (size 1.27 1.27)) hide)
     )
-    (property "LCSC" "C557685" (id 4) (at 204.47 71.12 0)
+    (property "LCSC" "C8404" (id 4) (at 204.47 71.12 0)
       (effects (font (size 1.27 1.27)) hide)
     )
@@
       (effects (font (size 1.27 1.27)) hide)
     )
-    (property "LCSC" "C557685" (id 4) (at 204.47 93.98 0)
+    (property "LCSC" "C8404" (id 4) (at 204.47 93.98 0)
       (effects (font (size 1.27 1.27)) hide)
     )
@@
       (effects (font (size 1.27 1.27)) hide)
     )
-    (property "LCSC" "C557685" (id 4) (at 227.33 86.36 0)
+    (property "LCSC" "C8404" (id 4) (at 227.33 86.36 0)
       (effects (font (size 1.27 1.27)) hide)
     )
@@
       (effects (font (size 1.27 1.27)) hide)
     )
-    (property "LCSC" "C557685" (id 4) (at 227.33 154.94 0)
+    (property "LCSC" "C8404" (id 4) (at 227.33 154.94 0)
       (effects (font (size 1.27 1.27)) hide)
     )
@@
       (effects (font (size 1.27 1.27)) hide)
     )
-    (property "LCSC" "C557685" (id 4) (at 204.47 48.26 0)
+    (property "LCSC" "C8404" (id 4) (at 204.47 48.26 0)
       (effects (font (size 1.27 1.27)) hide)
     )
@@
       (effects (font (size 1.27 1.27)) hide)
     )
-    (property "LCSC" "C557685" (id 4) (at 204.47 109.22 0)
+    (property "LCSC" "C8404" (id 4) (at 204.47 109.22 0)
       (effects (font (size 1.27 1.27)) hide)
     )
@@
       (effects (font (size 1.27 1.27)) hide)
     )
-    (property "LCSC" "C557685" (id 4) (at 204.47 116.84 0)
+    (property "LCSC" "C8404" (id 4) (at 204.47 116.84 0)
       (effects (font (size 1.27 1.27)) hide)
     )
@@
       (effects (font (size 1.27 1.27)) hide)
     )
-    (property "LCSC" "C557685" (id 4) (at 227.33 81.28 0)
+    (property "LCSC" "C8404" (id 4) (at 227.33 81.28 0)
       (effects (font (size 1.27 1.27)) hide)
     )
@@
       (effects (font (size 1.27 1.27)) hide)
     )
-    (property "LCSC" "C557685" (id 4) (at 204.47 142.24 0)
+    (property "LCSC" "C8404" (id 4) (at 204.47 142.24 0)
       (effects (font (size 1.27 1.27)) hide)
     )
@@
       (effects (font (size 1.27 1.27)) hide)
     )
-    (property "LCSC" "C557685" (id 4) (at 227.33 71.12 0)
+    (property "LCSC" "C8404" (id 4) (at 227.33 71.12 0)
       (effects (font (size 1.27 1.27)) hide)
     )
@@
       (effects (font (size 1.27 1.27)) hide)
     )
-    (property "LCSC" "C557685" (id 4) (at 227.33 149.86 0)
+    (property "LCSC" "C8404" (id 4) (at 227.33 149.86 0)
       (effects (font (size 1.27 1.27)) hide)
     )
@@
       (effects (font (size 1.27 1.27)) hide)
     )
-    (property "LCSC" "C557685" (id 4) (at 227.33 76.2 0)
+    (property "LCSC" "C8404" (id 4) (at 227.33 76.2 0)
       (effects (font (size 1.27 1.27)) hide)
     )
@@
       (effects (font (size 1.27 1.27)) hide)
     )
-    (property "LCSC" "C557685" (id 4) (at 227.33 116.84 0)
+    (property "LCSC" "C8404" (id 4) (at 227.33 116.84 0)
       (effects (font (size 1.27 1.27)) hide)
     )
@@
       (effects (font (size 1.27 1.27)) hide)
     )
-    (property "LCSC" "C557685" (id 4) (at 227.33 127 0)
+    (property "LCSC" "C8404" (id 4) (at 227.33 127 0)
       (effects (font (size 1.27 1.27)) hide)
     )
@@
       (effects (font (size 1.27 1.27)) hide)
     )
-    (property "LCSC" "C557685" (id 4) (at 227.33 121.92 0)
+    (property "LCSC" "C8404" (id 4) (at 227.33 121.92 0)
       (effects (font (size 1.27 1.27)) hide)
     )
@@
       (effects (font (size 1.27 1.27)) hide)
     )
-    (property "LCSC" "C557685" (id 4) (at 227.33 53.34 0)
+    (property "LCSC" "C8404" (id 4) (at 227.33 53.34 0)
       (effects (font (size 1.27 1.27)) hide)
     )
@@
       (effects (font (size 1.27 1.27)) hide)
     )
-    (property "LCSC" "C557685" (id 4) (at 204.47 127 0)
+    (property "LCSC" "C8404" (id 4) (at 204.47 127 0)
       (effects (font (size 1.27 1.27)) hide)
     )
@@
       (effects (font (size 1.27 1.27)) hide)
     )
-    (property "LCSC" "C557685" (id 4) (at 271.78 114.3 0)
+    (property "LCSC" "C8404" (id 4) (at 271.78 114.3 0)
       (effects (font (size 1.27 1.27)) hide)
     )
@@
       (effects (font (size 1.27 1.27)) hide)
     )
-    (property "LCSC" "C557685" (id 4) (at 204.47 76.2 0)
+    (property "LCSC" "C8404" (id 4) (at 204.47 76.2 0)
       (effects (font (size 1.27 1.27)) hide)
     )
@@
       (effects (font (size 1.27 1.27)) hide)
     )
-    (property "LCSC" "C557685" (id 4) (at 204.47 104.14 0)
+    (property "LCSC" "C8404" (id 4) (at 204.47 104.14 0)
       (effects (font (size 1.27 1.27)) hide)
     )
@@
       (effects (font (size 1.27 1.27)) hide)
     )
-    (property "LCSC" "C557685" (id 4) (at 204.47 147.32 0)
+    (property "LCSC" "C8404" (id 4) (at 204.47 147.32 0)
       (effects (font (size 1.27 1.27)) hide)
     )
@@
       (effects (font (size 1.27 1.27)) hide)
     )
-    (property "LCSC" "C557685" (id 4) (at 227.33 99.06 0)
+    (property "LCSC" "C8404" (id 4) (at 227.33 99.06 0)
       (effects (font (size 1.27 1.27)) hide)
     )
@@
       (effects (font (size 1.27 1.27)) hide)
     )
-    (property "LCSC" "C557685" (id 4) (at 227.33 132.08 0)
+    (property "LCSC" "C8404" (id 4) (at 227.33 132.08 0)
       (effects (font (size 1.27 1.27)) hide)
     )
@@
       (effects (font (size 1.27 1.27)) hide)
     )
-    (property "LCSC" "C557685" (id 4) (at 204.47 81.28 0)
+    (property "LCSC" "C8404" (id 4) (at 204.47 81.28 0)
       (effects (font (size 1.27 1.27)) hide)
     )
@@
       (effects (font (size 1.27 1.27)) hide)
     )
-    (property "LCSC" "C557685" (id 4) (at 204.47 132.08 0)
+    (property "LCSC" "C8404" (id 4) (at 204.47 132.08 0)
       (effects (font (size 1.27 1.27)) hide)
     )
@@
       (effects (font (size 1.27 1.27)) hide)
     )
-    (property "LCSC" "C557685" (id 4) (at 227.33 48.26 0)
+    (property "LCSC" "C8404" (id 4) (at 227.33 48.26 0)
       (effects (font (size 1.27 1.27)) hide)
     )
@@
       (effects (font (size 1.27 1.27)) hide)
     )
-    (property "LCSC" "C557685" (id 4) (at 204.47 53.34 0)
+    (property "LCSC" "C8404" (id 4) (at 204.47 53.34 0)
       (effects (font (size 1.27 1.27)) hide)
     )
@@
       (effects (font (size 1.27 1.27)) hide)
     )
-    (property "LCSC" "C557685" (id 4) (at 227.33 93.98 0)
+    (property "LCSC" "C8404" (id 4) (at 227.33 93.98 0)
       (effects (font (size 1.27 1.27)) hide)
     )
@@
       (effects (font (size 1.27 1.27)) hide)
     )
-    (property "LCSC" "C557685" (id 4) (at 204.47 99.06 0)
-      (effects (font (size 1.27 1.27)) hide)
-    )
+    (property "LCSC" "C8404" (id 4) (at 204.47 99.06 0)
+      (effects (font (size 1.27 1.27)) hide)
+    )
