File: PCBs/Slaves/Nano SFF Slave/Nano SFF Slave.kicad_pcb (KiCad board)
At the start: 2 copper layers, 52.4 x 50 mm, 52 parts, among them J1 Screw_Terminal_01x02, J10 AVR-ISP-6, J11 Conn_01x06_Female, J12 Screw_Terminal_01x02, J13 Screw_Terminal_01x02, J14 Screw_Terminal_01x02, J15 Screw_Terminal_01x02, J16 Screw_Terminal_01x02, J2 Screw_Terminal_01x02, J3 Screw_Terminal_01x02, J4 Screw_Terminal_01x02, J5 Screw_Terminal_01x02, J6 Screw_Terminal_01x02, J7 Screw_Terminal_01x02, J8 Screw_Terminal_01x02, J9 Screw_Terminal_01x02, SW1 SW_DIP_x02, SW2 SW_DIP_x02, SW3 SW_MEC_5E, U1 ATmega328P-AU, U2 MAX487ESA+T, U3 ULN2003A, U4 MAX487CPA+, U5 AMS1117-5.0, Y1 Crystal_GND24

Commit message: Cleaned up PCB
Parts:
- moved REF** 0.45 mm to (120.8, 107.1)
Changed lines of the file:
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@@
     (fp_line (start 1 -0.625) (end 1 0.625) (layer "F.Fab") (width 0.1))
     (fp_line (start 1 0.625) (end -1 0.625) (layer "F.Fab") (width 0.1))
-    (pad "1" smd roundrect (at -0.9125 0) (size 1.025 1.4) (layers "F.Cu" "F.Paste" "F.Mask") (roundrect_rratio 0.243902)
+    (pad "1" smd roundrect (at -0.9125 0) (size 1.025 1.4) (layers "F.Cu" "F.Paste" "F.Mask") (roundrect_rratio 0.243902439)
       (net 45 "Net-(SW1-Pad4)") (pintype "passive"))
-    (pad "2" smd roundrect (at 0.9125 0) (size 1.025 1.4) (layers "F.Cu" "F.Paste" "F.Mask") (roundrect_rratio 0.243902)
+    (pad "2" smd roundrect (at 0.9125 0) (size 1.025 1.4) (layers "F.Cu" "F.Paste" "F.Mask") (roundrect_rratio 0.243902439)
       (net 9 "D2") (pintype "passive"))
     (model "${KICAD6_3DMODEL_DIR}/Resistor_SMD.3dshapes/R_0805_2012Metric.wrl"
@@
   )
   (footprint "Symbol:OSHW-Logo2_7.3x6mm_Copper" (layer "F.Cu")
-    (at 120.65 106.68)
+    (at 120.824192 107.090338)
     (descr "Open Source Hardware Symbol")
     (tags "Logo Symbol OSHW")
@@
     (effects (font (size 0.8128 0.8128) (thickness 0.1524)))
   )
-  (gr_text "${TITLE} Rev. ${REVISION}" (at 153.982521 103.52826 90) (layer "F.SilkS")
+  (gr_text "${TITLE} Rev. ${REVISION}" (at 153.628292 103.52826 90) (layer "F.SilkS")
     (effects (font (size 0.8128 0.8128) (thickness 0.127)) (justify right))
   )
@@
     (effects (font (size 0.8128 0.8128) (thickness 0.1524)))
   )
-  (gr_text "WarthogAtHome.com" (at 153.982521 84.72591 90) (layer "F.SilkS")
+  (gr_text "WarthogAtHome.com" (at 153.628292 84.72591 90) (layer "F.SilkS")
     (effects (font (size 0.6096 0.6096) (thickness 0.1016)) (justify right))
   )
@@
   (segment (start 149.111493 103.167888) (end 148.349592 103.167888) (width 0.1524) (layer "B.Cu") (net 3))
   (segment (start 148.349592 103.167888) (end 145.227242 106.290238) (width 0.1524) (layer "B.Cu") (net 3))
-  (segment (start 145.227242 89.888188) (end 145.227242 83.487388) (width 0.1524) (layer "B.Cu") (net 3))
+  (segment (start 145.227242 93.966738) (end 145.227242 83.487388) (width 0.1524) (layer "B.Cu") (net 3))
   (segment (start 145.227242 106.290238) (end 145.227242 103.489888) (width 0.1524) (layer "B.Cu") (net 3))
   (segment (start 145.227242 103.489888) (end 144.427142 102.689788) (width 0.1524) (layer "B.Cu") (net 3))
@@
   (segment (start 145.227242 83.487388) (end 146.427392 82.287238) (width 0.1524) (layer "B.Cu") (net 3))
   (segment (start 149.107071 103.163466) (end 149.107071 100.48256) (width 0.1524) (layer "B.Cu") (net 3))
-  (segment (start 145.227242 93.966738) (end 145.227242 89.888188) (width 0.1524) (layer "B.Cu") (net 3))
   (segment (start 142.680315 96.659688) (end 142.681907 96.66128) (width 0.1524) (layer "F.Cu") (net 4))
   (segment (start 138.902242 91.564188) (end 138.902242 90.663288) (width 0.1524) (layer "F.Cu") (net 4))
@@
   (via (at 139.626542 109.890688) (size 0.5) (drill 0.2) (layers "F.Cu" "B.Cu") (net 10))
   (segment (start 139.626542 109.890688) (end 134.425892 109.890688) (width 0.1524) (layer "B.Cu") (net 10))
-  (segment (start 134.025842 110.290738) (end 129.225242 115.091338) (width 0.1524) (layer "B.Cu") (net 10))
-  (segment (start 134.425892 109.890688) (end 134.025842 110.290738) (width 0.1524) (layer "B.Cu") (net 10))
+  (segment (start 129.225242 115.091338) (end 134.425892 109.890688) (width 0.1524) (layer "B.Cu") (net 10))
   (segment (start 140.426742 109.890588) (end 139.626542 110.690788) (width 0.1524) (layer "F.Cu") (net 11))
   (segment (start 130.025342 115.091338) (end 122.424392 122.692288) (width 0.1524) (layer "F.Cu") (net 11))
@@
   (via (at 147.948842 120.291988) (size 0.5) (drill 0.2) (layers "F.Cu" "B.Cu") (net 18))
   (segment (start 153.306292 98.689288) (end 152.750142 98.689288) (width 0.1524) (layer "B.Cu") (net 18))
-  (segment (start 153.228242 120.291988) (end 153.628292 119.891938) (width 0.1524) (layer "B.Cu") (net 18))
   (segment (start 147.948842 120.291988) (end 153.228242 120.291988) (width 0.1524) (layer "B.Cu") (net 18))
-  (segment (start 153.628292 119.891938) (end 153.706441 119.813789) (width 0.1524) (layer "B.Cu") (net 18))
+  (segment (start 153.228242 120.291988) (end 153.706441 119.813789) (width 0.1524) (layer "B.Cu") (net 18))
   (segment (start 153.706342 99.089338) (end 153.306292 98.689288) (width 0.1524) (layer "B.Cu") (net 18))
   (segment (start 153.706441 119.813789) (end 153.706441 118.026064) (width 0.1524) (layer "B.Cu") (net 18))
@@
   (segment (start 143.226992 95.166888) (end 140.990421 97.403459) (width 0.1524) (layer "F.Cu") (net 28))
   (segment (start 138.579068 103.642564) (end 136.693502 101.756998) (width 0.1524) (layer "F.Cu") (net 28))
-  (segment (start 121.701394 101.812586) (end 127.582879 101.812586) (width 0.1524) (layer "F.Cu") (net 28))
   (segment (start 140.990421 97.403459) (end 140.990421 97.92756) (width 0.1524) (layer "F.Cu") (net 28))
   (segment (start 136.693502 101.756998) (end 132.558332 101.756998) (width 0.1524) (layer "F.Cu") (net 28))
@@
   (segment (start 144.426942 107.640588) (end 144.426942 106.290438) (width 0.1524) (layer "F.Cu") (net 28))
   (segment (start 139.885526 103.642564) (end 138.579068 103.642564) (width 0.1524) (layer "F.Cu") (net 28))
-  (segment (start 121.701394 101.812586) (end 121.14714 101.812586) (width 0.1524) (layer "F.Cu") (net 28))
+  (segment (start 121.14714 101.812586) (end 127.582879 101.812586) (width 0.1524) (layer "F.Cu") (net 28))
   (segment (start 127.582879 101.812586) (end 127.63892 101.756545) (width 0.1524) (layer "F.Cu") (net 28))
   (segment (start 144.426942 106.290438) (end 144.427142 106.290238) (width 0.1524) (layer "F.Cu") (net 28))
@@
   (segment (start 120.758842 99.489388) (end 118.758592 97.489138) (width 0.1524) (layer "B.Cu") (net 34))
   (segment (start 114.455483 97.203657) (end 110.49 97.203657) (width 0.1524) (layer "B.Cu") (net 34))
-  (segment (start 124.824692 100.689538) (end 123.624542 99.489388) (width 0.1524) (layer "B.Cu") (net 34))
+  (segment (start 123.624542 99.489388) (end 126.883462 102.748308) (width 0.1524) (layer "B.Cu") (net 34))
   (segment (start 114.463796 97.21197) (end 114.455483 97.203657) (width 0.1524) (layer "B.Cu") (net 34))
-  (segment (start 121.624292 99.489388) (end 120.758842 99.489388) (width 0.1524) (layer "B.Cu") (net 34))
   (segment (start 128.766672 102.748308) (end 126.883462 102.748308) (width 0.1524) (layer "B.Cu") (net 34))
-  (segment (start 123.624542 99.489388) (end 121.624292 99.489388) (width 0.1524) (layer "B.Cu") (net 34))
-  (segment (start 126.883462 102.748308) (end 124.824692 100.689538) (width 0.1524) (layer "B.Cu") (net 34))
+  (segment (start 120.758842 99.489388) (end 123.624542 99.489388) (width 0.1524) (layer "B.Cu") (net 34))
   (segment (start 144.427142 123.092338) (end 143.739968 123.779512) (width 0.1524) (layer "F.Cu") (net 35))
   (segment (start 143.739968 123.779512) (end 143.739968 126.981223) (width 0.1524) (layer "F.Cu") (net 35))
@@
   (via (at 151.628042 117.891688) (size 0.5) (drill 0.2) (layers "F.Cu" "B.Cu") (net 36))
   (via (at 151.144492 110.658706) (size 0.5) (drill 0.2) (layers "F.Cu" "B.Cu") (net 36))
-  (segment (start 151.628042 111.142256) (end 151.628042 111.490888) (width 0.1524) (layer "B.Cu") (net 36))
   (segment (start 151.144492 110.658706) (end 151.628042 111.142256) (width 0.1524) (layer "B.Cu") (net 36))
-  (segment (start 151.628042 111.490888) (end 151.628042 117.891688) (width 0.1524) (layer "B.Cu") (net 36))
+  (segment (start 151.628042 111.142256) (end 151.628042 117.891688) (width 0.1524) (layer "B.Cu") (net 36))
   (segment (start 119.650363 117.424204) (end 123.291926 117.424204) (width 0.2032) (layer "F.Cu") (net 37))
   (segment (start 122.024342 118.691788) (end 122.021924 118.694206) (width 0.2032) (layer "F.Cu") (net 37))
