File: PCBs/Slaves/Mega SFF Slave/Mega SFF Slave.kicad_pcb (KiCad board)
At the start: 2 copper layers, 87.1 x 57 mm, 80 parts, among them J1 AVR-ISP-6, J10 Screw_Terminal_01x02, J11 Screw_Terminal_01x02, J12 Screw_Terminal_01x02, J13 Screw_Terminal_01x02, J14 Screw_Terminal_01x02, J15 Screw_Terminal_01x02, J16 Screw_Terminal_01x02, J17 Screw_Terminal_01x02, J18 Screw_Terminal_01x02, J19 Screw_Terminal_01x02, J2 Screw_Terminal_01x02, J20 Screw_Terminal_01x02, J21 Screw_Terminal_01x02, J22 Screw_Terminal_01x02, J23 Screw_Terminal_01x02, J24 Screw_Terminal_01x02, J25 Screw_Terminal_01x02, J26 Screw_Terminal_01x02, J27 Screw_Terminal_01x02, J28 Screw_Terminal_01x02, J29 Screw_Terminal_01x02, J3 Screw_Terminal_01x02, J30 Screw_Terminal_01x02, J31 Screw_Terminal_01x02, J32 Screw_Terminal_01x02, J33 Screw_Terminal_01x02, J34 Screw_Terminal_01x02, J35 Screw_Terminal_01x02, J36 Screw_Terminal_01x02, J37 Screw_Terminal_01x02, J39 Conn_01x06_Female, J4 Screw_Terminal_01x02, J40 Screw_Terminal_01x02, J41 Screw_Terminal_01x02, J5 Screw_Terminal_01x02, J6 Screw_Terminal_01x02, J7 Screw_Terminal_01x02, J8 Screw_Terminal_01x02, J9 Screw_Terminal_01x02, SW1 SW_MEC_5E, SW2 SW_DIP_x02, SW3 SW_DIP_x02, U1 ATmega2560-16A, U2 MAX487ESA+T, U3 AMS1117-5.0, U4 ULN2003A, U5 MAX487ESA+T, Y1 Crystal_GND24

Commit message: Mega SFF Slave WIP
Parts:
- moved C9 2.75 mm to (110.5, 88.5), turned to 180 degrees
- moved C2 0.25 mm to (140.8, 95.5)
- turned C6 to 0 degrees
Routing:
- net +5V: track 0.00 -> 120.2 mm, vias 0 -> 6
- net +12V: track 0.00 -> 2.05 mm
- removed copper zone on F.Cu, net +12V
Changed lines of the file:
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@@
     )
     (pad_to_mask_clearance 0)
+    (grid_origin 124.550997 87.974665)
     (pcbplotparams
       (layerselection 0x00010fc_ffffffff)
@@
   )
   (footprint "A10 KiCad Libraries:C0402" (layer "F.Cu")
-    (at 136.309215 83.16197 180)
+    (at 136.309215 83.16197)
     (descr "C0402 footprint")
     (tags "C0402 footprint")
@@
     (property "Sheetname" "")
     (attr through_hole)
-    (fp_text reference "C6" (at 0 -1.160695) (layer "F.SilkS")
+    (fp_text reference "C6" (at 0 1.312695) (layer "F.SilkS")
       (effects (font (size 0.5588 0.5588) (thickness 0.1016)))
     )
@@
     (fp_line (start -1.27 -0.635) (end 1.27 -0.635) (layer "F.CrtYd") (width 0.1))
     (fp_line (start 1.27 0.635) (end -1.27 0.635) (layer "F.CrtYd") (width 0.1))
-    (pad "1" smd rect (at -0.545085 0 180) (size 0.790094 0.540005) (layers "F.Cu" "F.Paste" "F.Mask")
+    (pad "1" smd rect (at -0.545085 0) (size 0.790094 0.540005) (layers "F.Cu" "F.Paste" "F.Mask")
       (net 1 "+5V") (pintype "passive"))
-    (pad "2" smd rect (at 0.545085 0 180) (size 0.790094 0.540005) (layers "F.Cu" "F.Paste" "F.Mask")
+    (pad "2" smd rect (at 0.545085 0) (size 0.790094 0.540005) (layers "F.Cu" "F.Paste" "F.Mask")
       (net 2 "GND") (pintype "passive"))
     (model ":WarthogAtHome:C0402.wrl"
@@
   )
   (footprint "A10 KiCad Libraries:C0402" (layer "F.Cu")
-    (at 107.75 88.5)
+    (at 110.5 88.5 180)
     (descr "C0402 footprint")
     (tags "C0402 footprint")
@@
     (fp_line (start -1.27 0.635) (end -1.27 -0.635) (layer "F.CrtYd") (width 0.1))
     (fp_line (start -1.27 -0.635) (end 1.27 -0.635) (layer "F.CrtYd") (width 0.1))
-    (pad "1" smd rect (at -0.545085 0) (size 0.790094 0.540005) (layers "F.Cu" "F.Paste" "F.Mask")
+    (pad "1" smd rect (at -0.545085 0 180) (size 0.790094 0.540005) (layers "F.Cu" "F.Paste" "F.Mask")
       (net 1 "+5V") (pintype "passive"))
-    (pad "2" smd rect (at 0.545085 0) (size 0.790094 0.540005) (layers "F.Cu" "F.Paste" "F.Mask")
+    (pad "2" smd rect (at 0.545085 0 180) (size 0.790094 0.540005) (layers "F.Cu" "F.Paste" "F.Mask")
       (net 2 "GND") (pintype "passive"))
     (model ":WarthogAtHome:C0402.wrl"
@@
   )
   (footprint "A10 KiCad Libraries:C0402" (layer "F.Cu")
-    (at 141.050997 95.474665)
+    (at 140.800997 95.474665)
     (descr "C0402 footprint")
     (tags "C0402 footprint")
@@
     (effects (font (size 1.2192 1.2192) (thickness 0.2032)))
   )
+  (segment (start 136.550997 101.637165) (end 137.463497 101.637165) (width 0.1778) (layer "F.Cu") (net 1))
+  (segment (start 135.300997 84.224665) (end 134.300997 84.224665) (width 0.1778) (layer "F.Cu") (net 1))
+  (segment (start 140.255912 96.01975) (end 139.800997 96.474665) (width 0.1778) (layer "F.Cu") (net 1))
+  (segment (start 137.463497 101.637165) (end 137.550997 101.724665) (width 0.1778) (layer "F.Cu") (net 1))
+  (segment (start 138.213497 95.474665) (end 140.255912 95.474665) (width 0.1778) (layer "F.Cu") (net 1))
+  (segment (start 135.76413 83.16197) (end 135.76413 84.187798) (width 0.1778) (layer "F.Cu") (net 1))
+  (segment (start 135.76413 84.187798) (end 135.800997 84.224665) (width 0.1778) (layer "F.Cu") (net 1))
+  (segment (start 135.800997 84.224665) (end 135.300997 84.224665) (width 0.1778) (layer "F.Cu") (net 1))
+  (segment (start 121.050997 92.864082) (end 121.050997 93.974665) (width 0.1778) (layer "F.Cu") (net 1))
+  (segment (start 140.255912 95.474665) (end 140.255912 96.01975) (width 0.1778) (layer "F.Cu") (net 1))
+  (segment (start 108.995 84.055) (end 110.555 84.055) (width 0.8128) (layer "F.Cu") (net 1))
+  (segment (start 121.16158 92.974665) (end 121.050997 92.864082) (width 0.1778) (layer "F.Cu") (net 1))
+  (segment (start 111.045085 88.5) (end 111.045085 84.545085) (width 0.8128) (layer "F.Cu") (net 1))
+  (segment (start 138.895912 101.637165) (end 137.638497 101.637165) (width 0.1778) (layer "F.Cu") (net 1))
+  (segment (start 122.888497 92.974665) (end 121.16158 92.974665) (width 0.1778) (layer "F.Cu") (net 1))
+  (segment (start 134.050997 86.312165) (end 134.050997 89.474665) (width 0.1778) (layer "F.Cu") (net 1))
+  (segment (start 139.800997 84.224665) (end 135.800997 84.224665) (width 0.1778) (layer "F.Cu") (net 1))
+  (segment (start 111.550997 89.474665) (end 112.800997 89.474665) (width 0.8128) (layer "F.Cu") (net 1))
+  (segment (start 125.050997 103.474665) (end 126.550997 103.474665) (width 0.8128) (layer "F.Cu") (net 1))
+  (segment (start 134.050997 84.474665) (end 134.050997 86.312165) (width 0.1778) (layer "F.Cu") (net 1))
+  (segment (start 111.045085 88.968753) (end 111.550997 89.474665) (width 0.8128) (layer "F.Cu") (net 1))
+  (segment (start 111.045085 88.5) (end 111.045085 88.968753) (width 0.8128) (layer "F.Cu") (net 1))
+  (segment (start 140.050997 83.974665) (end 139.800997 84.224665) (width 0.1778) (layer "F.Cu") (net 1))
+  (segment (start 134.300997 84.224665) (end 134.050997 84.474665) (width 0.1778) (layer "F.Cu") (net 1))
+  (segment (start 111.045085 84.545085) (end 110.555 84.055) (width 0.8128) (layer "F.Cu") (net 1))
+  (segment (start 140.050997 83.258198) (end 140.050997 83.974665) (width 0.1778) (layer "F.Cu") (net 1))
+  (segment (start 137.638497 101.637165) (end 137.550997 101.724665) (width 0.1778) (layer "F.Cu") (net 1))
+  (via (at 137.550997 101.724665) (size 0.8128) (drill 0.4064) (layers "F.Cu" "B.Cu") (net 1))
+  (via (at 121.050997 93.974665) (size 0.8128) (drill 0.4064) (layers "F.Cu" "B.Cu") (net 1))
+  (via (at 139.800997 96.474665) (size 0.8128) (drill 0.4064) (layers "F.Cu" "B.Cu") (net 1))
+  (via (at 134.050997 89.474665) (size 0.8128) (drill 0.4064) (layers "F.Cu" "B.Cu") (net 1))
+  (via (at 112.800997 89.474665) (size 0.8128) (drill 0.4064) (layers "F.Cu" "B.Cu") (net 1))
+  (via (at 125.050997 103.474665) (size 0.8128) (drill 0.4064) (layers "F.Cu" "B.Cu") (net 1))
+  (segment (start 149.270494 101.718494) (end 137.557168 101.718494) (width 0.1778) (layer "B.Cu") (net 1))
+  (segment (start 145.420329 90.593997) (end 147.785997 90.593997) (width 0.8128) (layer "B.Cu") (net 1))
+  (segment (start 125.050997 94.724665) (end 125.050997 103.474665) (width 0.8128) (layer "B.Cu") (net 1))
+  (segment (start 137.550997 102.224665) (end 137.550997 101.224665) (width 0.8128) (layer "B.Cu") (net 1))
+  (segment (start 112.800997 89.474665) (end 120.550997 89.474665) (width 0.8128) (layer "B.Cu") (net 1))
+  (segment (start 138.300997 96.974665) (end 138.800997 96.474665) (width 0.8128) (layer "B.Cu") (net 1))
+  (segment (start 125.050997 103.474665) (end 137.050997 103.474665) (width 0.8128) (layer "B.Cu") (net 1))
+  (segment (start 150.845997 103.293997) (end 149.270494 101.718494) (width 0.1778) (layer "B.Cu") (net 1))
+  (segment (start 137.050997 103.474665) (end 137.550997 102.974665) (width 0.8128) (layer "B.Cu") (net 1))
+  (segment (start 133.550997 89.474665) (end 134.050997 89.474665) (width 0.8128) (layer "B.Cu") (net 1))
+  (segment (start 144.300997 89.474665) (end 145.420329 90.593997) (width 0.8128) (layer "B.Cu") (net 1))
+  (segment (start 138.800997 96.474665) (end 139.800997 96.474665) (width 0.8128) (layer "B.Cu") (net 1))
+  (segment (start 137.557168 101.718494) (end 137.550997 101.724665) (width 0.1778) (layer "B.Cu") (net 1))
+  (segment (start 138.050997 100.724665) (end 138.300997 100.474665) (width 0.8128) (layer "B.Cu") (net 1))
+  (segment (start 138.300997 100.474665) (end 138.300997 96.974665) (width 0.8128) (layer "B.Cu") (net 1))
+  (segment (start 124.300997 93.974665) (end 125.050997 94.724665) (width 0.8128) (layer "B.Cu") (net 1))
+  (segment (start 137.550997 101.224665) (end 138.050997 100.724665) (width 0.8128) (layer "B.Cu") (net 1))
+  (segment (start 134.050997 89.474665) (end 144.300997 89.474665) (width 0.8128) (layer "B.Cu") (net 1))
+  (segment (start 137.550997 102.224665) (end 137.550997 101.724665) (width 0.8128) (layer "B.Cu") (net 1))
+  (segment (start 120.550997 89.474665) (end 133.550997 89.474665) (width 0.8128) (layer "B.Cu") (net 1))
+  (segment (start 137.550997 102.974665) (end 137.550997 102.224665) (width 0.8128) (layer "B.Cu") (net 1))
+  (segment (start 121.050997 93.974665) (end 124.300997 93.974665) (width 0.8128) (layer "B.Cu") (net 1))
+  (segment (start 121.050997 89.974665) (end 121.050997 93.974665) (width 0.8128) (layer "B.Cu") (net 1))
+  (segment (start 120.550997 89.474665) (end 121.050997 89.974665) (width 0.8128) (layer "B.Cu") (net 1))
+  (segment (start 92.16352 90.678001) (end 90.382976 89.661999) (width 1.6256) (layer "F.Cu") (net 3))
   (zone (net 2) (net_name "GND") (layers F&B.Cu) (name "GND") (hatch edge 0.508)
     (connect_pads (clearance 0.1524))
@@
       )
     )
-  )
-  (zone (net 3) (net_name "+12V") (layer "F.Cu") (name "12V") (hatch edge 0.508)
-    (priority 10)
-    (connect_pads yes (clearance 0.1524))
-    (min_thickness 0.1524) (filled_areas_thickness no)
-    (fill (thermal_gap 0.508) (thermal_bridge_width 0.508) (smoothing fillet) (radius 0.8128))
-    (polygon
-      (pts
-        (xy 92.132157 91.499)
-        (xy 90.371441 90.522942)
-        (xy 89.483423 90.474915)
-        (xy 89.483423 88.795364)
-        (xy 92.130607 88.795301)
-      )
-    )

Commit message: Mega SFF WIP
Parts:
- moved REF** 29.9 mm to (142.3, 107.2)
- moved C14 13.7 mm to (155.6, 95.4), turned to -90 degrees
- moved C9 12.9 mm to (101.1, 79.7), turned to -90 degrees
- moved J39 12.3 mm to (153.1, 96.0), turned to 0 degrees
- moved D3 10.6 mm to (159.1, 107.0)
- moved R7 10.6 mm to (157.1, 107.0)
- moved C8 10.2 mm to (108.1, 89.0), turned to -90 degrees
- moved R2 7.36 mm to (100.3, 97.5), turned to 90 degrees
- moved J1 5.00 mm to (151.6, 85.7)
- moved C7 2.88 mm to (113.1, 86.2), turned to 90 degrees
- moved U3 2.58 mm to (105.8, 81.5), turned to 90 degrees
- moved R6 2.31 mm to (98.1, 79.7), turned to -90 degrees
- moved C5 1.67 mm to (120.8, 94.0), turned to -45 degrees
- moved D2 1.50 mm to (95.3, 80.6)
- moved R4 1.41 mm to (100.3, 93.2)
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Routing:
- net D13: track 0.00 -> 95.0 mm, vias 0 -> 4
- net TXD: track 0.00 -> 74.7 mm, vias 0 -> 5
- net RXD: track 0.00 -> 73.7 mm, vias 0 -> 5
- net D4: track 0.00 -> 72.7 mm, vias 0 -> 4
- net +12V: track 2.05 -> 68.9 mm, vias 0 -> 1
- net D22: track 0.00 -> 59.8 mm, vias 0 -> 2
- net RESET: track 0.00 -> 57.8 mm, vias 0 -> 2
- net D23: track 0.00 -> 56.6 mm, vias 0 -> 2
- net D24: track 0.00 -> 53.2 mm, vias 0 -> 2
- net A15: track 0.00 -> 51.1 mm
- net D19: track 0.00 -> 50.4 mm, vias 0 -> 2
- net +5V: track 120.2 -> 169.7 mm, vias 6 -> 39
- net A14: track 0.00 -> 48.9 mm
- net D20: track 0.00 -> 48.1 mm, vias 0 -> 2
- net D39: track 0.00 -> 46.8 mm, vias 0 -> 2
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- added copper zone on B.Cu, net +5V
- added copper zone on F.Cu, net +5V

Commit message: Mega SFF Slave Rev. 1
Other:
- board text added: "50MM"
- board text added: "80MM"
