File: PCBs/Master/Standalone/Master.kicad_pcb (KiCad board)
At the start: 2 copper layers, 82.8 x 55.2 mm, 32 parts

Commit message: Master WIP
Parts:
- removed F1: 6A, A10 KiCad Libraries:FUSE_BK-6013
- removed HOLE-1, HOLE-2, HOLE-3, HOLE-4: MountingHole_3.2mm_M3, MountingHole:MountingHole_3.2mm_M3
- removed MASTER-1, MASTER-2, MASTER-3: MAX487CPA+, Package_DIP:DIP-8_W7.62mm_LongPads
- removed MEGA-1, MEGA-2: Conn_01x06_Male, A10 KiCad Libraries:SHDR6W64P0X250_1X6_1740X575X700P
- added C12: 100nF, A10 KiCad Libraries:C0402, F.Cu at (100.0, 22.3)
- added C13: 10uF, A10 KiCad Libraries:C0402, F.Cu at (122.7, -2.71)
- added C14: 1uF, A10 KiCad Libraries:C0402, F.Cu at (104.0, 19.7)
- added C15: 15pF, A10 KiCad Libraries:C0402, F.Cu at (113.2, 9.40)
- added C16: 15pF, A10 KiCad Libraries:C0402, F.Cu at (119.4, 2.07)
- added C17: 1uF, A10 KiCad Libraries:C0402, F.Cu at (114.3, 72.5)
- added C18: 1uF, A10 KiCad Libraries:C0402, F.Cu at (170.3, 40.9)
- added C19: 1uF, A10 KiCad Libraries:C0402, F.Cu at (174.5, 4.76)
- added C4: 1uF, A10 KiCad Libraries:C0402, F.Cu at (104.4, 16.0)
- added C5: 1uF, A10 KiCad Libraries:C0402, F.Cu at (119.4, -0.30)
- added C6: 1uF, A10 KiCad Libraries:C0402, F.Cu at (111.6, 12.0)
- added C7: 100nF, A10 KiCad Libraries:C0402, F.Cu at (126.4, -2.71)
- added C8: 100nF, A10 KiCad Libraries:C0402, F.Cu at (126.8, -5.30)
- added D10: SM712_SOT23, Package_TO_SOT_SMD:SOT-23, F.Cu at (170.2, 2.01)
- added D11: BLUE, LED_SMD:LED_0603_1608Metric, F.Cu at (185.4, -8.14)
- added D5: LED, LED_SMD:LED_0603_1608Metric, F.Cu at (109.4, 9.51)
- added D6: SM712_SOT23, Package_TO_SOT_SMD:SOT-23, F.Cu at (124.8, 78.7)
- added D7: BLUE, LED_SMD:LED_0603_1608Metric, F.Cu at (147.8, 73.2)
- added D8: SM712_SOT23, Package_TO_SOT_SMD:SOT-23, F.Cu at (166.0, 38.2)
- added D9: BLUE, LED_SMD:LED_0603_1608Metric, F.Cu at (181.1, 28.0)
- added F10: 5A, A10 KiCad Libraries:FUSE_BK-6013, F.Cu at (143.8, 12.3)
- added F4: 5A, A10 KiCad Libraries:FUSE_BK-6013, F.Cu at (157.8, 78.7)
- added F5: 100mA, Fuse:Fuse_0603_1608Metric, F.Cu at (181.1, 30.6)
- added F6: 100mA, Fuse:Fuse_0603_1608Metric, F.Cu at (170.5, 38.5)
- added F7: 5A, A10 KiCad Libraries:FUSE_BK-6013, F.Cu at (139.5, 48.4)
- added F8: 100mA, Fuse:Fuse_0603_1608Metric, F.Cu at (185.3, -5.59)
- added F9: 100mA, Fuse:Fuse_0603_1608Metric, F.Cu at (174.7, 2.32)
- added H1: MountingHole, MountingHole:MountingHole_3.2mm_M3, F.Cu at (94.2, 19.5)
- added H2: MountingHole, MountingHole:MountingHole_3.2mm_M3, F.Cu at (116.9, -5.46)
- added H3: MountingHole, MountingHole:MountingHole_3.2mm_M3, F.Cu at (113.6, 4.24)
- added H4: MountingHole, MountingHole:MountingHole_3.2mm_M3, F.Cu at (105.7, 4.24)
- added J1: Conn_01x06_Female, Connector_PinSocket_2.54mm:PinSocket_1x06_P2.54mm_Vertical, F.Cu at (93.8, -7.11)
- added J2: AVR-ISP-6, Connector_PinHeader_2.54mm:PinHeader_2x03_P2.54mm_Vertical, F.Cu at (108.1, -7.11)
- added J3: USB_B_Micro, A10 KiCad Libraries:MICRO-USB-SMD_U254-051T-4BHJ25-F2S, F.Cu at (88.1, 68.2)
- added R10: 3.3K, Resistor_SMD:R_0805_2012Metric, F.Cu at (154.3, 73.0)
- added R11: 120R, Resistor_SMD:R_0805_2012Metric, F.Cu at (165.8, 41.9)
- added R12: 3.3K, Resistor_SMD:R_0805_2012Metric, F.Cu at (161.2, 46.3)
- added R13: 120R, Resistor_SMD:R_0805_2012Metric, F.Cu at (170.0, 5.71)
- added R14: 3.3K, Resistor_SMD:R_0805_2012Metric, F.Cu at (165.5, 10.2)
- added R8: 1K, Resistor_SMD:R_0805_2012Metric, F.Cu at (85.9, 20.5)
- added R9: 120R, Resistor_SMD:R_0805_2012Metric, F.Cu at (121.6, 78.7)
- added SW1: SW_MEC_5E, A10 KiCad Libraries:SW-SMD_4P-L5.1-W5.1-P3.70-LS6.5-TL-2, F.Cu at (96.6, 11.7)
- added SW2: SW_DIP_x01, A10 KiCad Libraries:SW-SMD_DSHP02TSGER, F.Cu at (87.5, 14.0)
- added U10: TBU-CA065-200-WH, A10 KiCad Libraries:DIO-SMD_3P-L6.5-W4.0-BI, F.Cu at (135.6, 54.5)
- added U11: TBU-CA065-200-WH, A10 KiCad Libraries:DIO-SMD_3P-L6.5-W4.0-BI, F.Cu at (144.2, 54.5)
- added U12: TISP4240M3BJR-S, A10 KiCad Libraries:DO-214AA_L4.4-W3.6-LS5.3-BI, F.Cu at (175.3, 29.4)
- added U13: MAX487ESA+T, Package_DIP:DIP-8_W7.62mm, F.Cu at (149.8, 46.9)
- added U14: MAX487ESA+T, A10 KiCad Libraries:SOIC-8_L5.0-W4.0-P1.27-LS6.0-BL, F.Cu at (167.7, 31.4)
- added U15: TISP4240M3BJR-S, A10 KiCad Libraries:DO-214AA_L4.4-W3.6-LS5.3-BI, F.Cu at (175.3, 34.6)
- added U16: TBU-CA065-200-WH, A10 KiCad Libraries:DIO-SMD_3P-L6.5-W4.0-BI, F.Cu at (139.8, 18.4)
- added U17: TBU-CA065-200-WH, A10 KiCad Libraries:DIO-SMD_3P-L6.5-W4.0-BI, F.Cu at (148.4, 18.4)
- added U18: TISP4240M3BJR-S, A10 KiCad Libraries:DO-214AA_L4.4-W3.6-LS5.3-BI, F.Cu at (179.5, -6.80)
- added U19: MAX487ESA+T, Package_DIP:DIP-8_W7.62mm, F.Cu at (154.0, 10.8)
- added U2: ATmega2560-16A, Package_QFP:TQFP-100_14x14mm_P0.5mm, F.Cu at (91.8, 82.0)
- added U20: MAX487ESA+T, A10 KiCad Libraries:SOIC-8_L5.0-W4.0-P1.27-LS6.0-BL, F.Cu at (171.9, -4.82)
- added U21: TISP4240M3BJR-S, A10 KiCad Libraries:DO-214AA_L4.4-W3.6-LS5.3-BI, F.Cu at (179.5, -1.55)
- added U3: CH340C, A10 KiCad Libraries:SOP-16_L10.0-W3.9-P1.27-LS6.0-BL, F.Cu at (79.1, 13.2)
- added U4: TBU-CA065-200-WH, A10 KiCad Libraries:DIO-SMD_3P-L6.5-W4.0-BI, F.Cu at (127.7, 74.5)
- added U5: TBU-CA065-200-WH, A10 KiCad Libraries:DIO-SMD_3P-L6.5-W4.0-BI, F.Cu at (127.8, 83.0)
- added U6: TISP4240M3BJR-S, A10 KiCad Libraries:DO-214AA_L4.4-W3.6-LS5.3-BI, F.Cu at (134.1, 82.2)
- added U7: MAX487ESA+T, Package_DIP:DIP-8_W7.62mm, F.Cu at (111.8, 74.9)
- added U8: MAX487ESA+T, A10 KiCad Libraries:SOIC-8_L5.0-W4.0-P1.27-LS6.0-BL, F.Cu at (115.6, 78.7)
- added U9: TISP4240M3BJR-S, A10 KiCad Libraries:DO-214AA_L4.4-W3.6-LS5.3-BI, F.Cu at (134.1, 75.2)
- added Y1: Crystal_GND24, Crystal:Crystal_SMD_3225-4Pin_3.2x2.5mm, F.Cu at (98.7, 0.39)
- BUS1, BUS2, BUS3: footprint A10 KiCad Libraries:Molex 43045-0800 -> A10 KiCad Libraries:Molex Micro-Fit 3.0 43045-0812
- C1: value 0.1uF -> 4.7uF; footprint A10 KiCad Libraries:FA14 -> A10 KiCad Libraries:C0805
- C2, C3: value 0.1uF -> 1uF; footprint A10 KiCad Libraries:FA14 -> A10 KiCad Libraries:C0402
- D1, D2, D4: value GREEN -> LED; footprint LED_SMD:LED_1210_3225Metric_Pad1.42x2.65mm_HandSolder -> LED_SMD:LED_0603_1608Metric
- D3: value GREEN -> DIODE; footprint LED_SMD:LED_1210_3225Metric_Pad1.42x2.65mm_HandSolder -> A10 KiCad Libraries:SOD-123_L2.7-W1.6-LS3.7-RD-1
- F2, F3: value 6A -> 100mA; footprint A10 KiCad Libraries:FUSE_BK-6013 -> Fuse:Fuse_0603_1608Metric
- PSU1, PSU2, PSU3: footprint A10 KiCad Libraries:Molex 43045-0400 -> A10 KiCad Libraries:Molex Micro-Fit 3.0 43045-0400
- R1: value 120Ω -> 10K; footprint Resistor_THT:R_Axial_DIN0207_L6.3mm_D2.5mm_P7.62mm_Horizontal -> Resistor_SMD:R_0805_2012Metric
- R2, R3: value 120Ω -> 1K; footprint Resistor_THT:R_Axial_DIN0207_L6.3mm_D2.5mm_P7.62mm_Horizontal -> Resistor_SMD:R_0805_2012Metric
- R4, R5, R6: value 1.8K -> 1K; footprint Resistor_SMD:R_1210_3225Metric_Pad1.30x2.65mm_HandSolder -> Resistor_SMD:R_0805_2012Metric; moved to F.Cu
- R7: value 400R -> 1K; footprint Resistor_SMD:R_1210_3225Metric_Pad1.30x2.65mm_HandSolder -> Resistor_SMD:R_0805_2012Metric; moved to F.Cu
- moved D4 135.4 mm to (123.0, -5.19)
- moved R7 135.3 mm to (98.3, 4.09), turned to 0 degrees
- moved D3 129.8 mm to (76.2, 19.1)
- moved PSU3 122.3 mm to (160.9, -2.63)
- moved R5 120.8 mm to (123.1, -7.96), turned to 0 degrees
- moved D1 119.5 mm to (127.4, -8.14)
- moved R6 114.0 mm to (100.3, 17.0), turned to 0 degrees
- moved R3 111.5 mm to (79.7, 22.1)
- moved D2 102.0 mm to (100.2, 19.8)
- moved R4 100.0 mm to (81.5, 19.0), turned to 0 degrees
- moved C3 97.4 mm to (107.9, 13.0), turned to 0 degrees
- moved C2 95.1 mm to (123.1, -0.34), turned to 0 degrees
- moved R2 88.0 mm to (103.9, 13.3)
- moved PSU2 86.5 mm to (156.7, 33.5)
- moved C1 84.3 mm to (104.5, 10.0), turned to 0 degrees
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Connections:
- net +12V renamed Net-(F4-Pad1)
- BUS1 pad 1: 12V_Fused -> Net-(BUS1-Pad1)
- BUS1 pad 3: unconnected-(BUS1-Pad3) -> Net-(BUS1-Pad1)
- BUS1 pad 4: unconnected-(BUS1-Pad4) -> GND
- BUS1 pad 5: 12V_Fused -> Net-(BUS1-Pad1)
- BUS1 pad 7: RS485-1-B -> RS485-1-
- BUS1 pad 8: RS485-1-A -> RS485-1+
- BUS2 pad 1: /12V_2_Fused -> Net-(BUS2-Pad1)
- BUS2 pad 3: unconnected-(BUS2-Pad3) -> Net-(BUS2-Pad1)
- BUS2 pad 4: unconnected-(BUS2-Pad4) -> GND
- BUS2 pad 5: /12V_2_Fused -> Net-(BUS2-Pad1)
- BUS2 pad 7: RS485-2-B -> RS485-2-
- BUS2 pad 8: RS485-2-A -> RS485-2+
- BUS3 pad 1: /12V_3_Fused -> Net-(BUS3-Pad1)
- BUS3 pad 3: unconnected-(BUS3-Pad3) -> Net-(BUS3-Pad1)
- BUS3 pad 4: unconnected-(BUS3-Pad4) -> GND
- BUS3 pad 5: /12V_3_Fused -> Net-(BUS3-Pad1)
- BUS3 pad 7: RS485-3-B -> RS485-2-
- BUS3 pad 8: RS485-3-A -> RS485-2+
- C1 pad 1: GND -> +5V
- C1 pad 2: +5V -> GND
- C2 pad 1: GND -> +5V
- C2 pad 2: +5V -> GND
- C3 pad 1: GND -> +5V
- C3 pad 2: +5V -> GND
- D1 pad 1: unconnected-(D1-Pad1) -> GND
- D2 pad 1: unconnected-(D2-Pad1) -> GND
- D3 pad 1: unconnected-(D3-Pad1) -> Net-(C12-Pad2)
- D3 pad 2: Net-(D3-Pad2) -> +5V
- D4 pad 1: GND -> USB_TXD
- F2 pad 1: +12V_2 -> Net-(F2-Pad1)
- F2 pad 2: /12V_2_Fused -> Net-(D6-Pad2)
- F3 pad 1: +12V_3 -> Net-(D6-Pad1)
- F3 pad 2: /12V_3_Fused -> Net-(F3-Pad2)
- PSU2 pad 2: +12V_2 -> Net-(F7-Pad1)
- PSU2 pad 4: +12V_2 -> Net-(F7-Pad1)
- PSU3 pad 2: +12V_3 -> Net-(F10-Pad1)
- PSU3 pad 4: +12V_3 -> Net-(F10-Pad1)
- R1 pad 1: RS485-1-B -> +5V
- R1 pad 2: RS485-1-A -> RESET
- R2 pad 1: RS485-2-B -> D13
- R2 pad 2: RS485-2-A -> Net-(D1-Pad2)
- R3 pad 1: RS485-3-B -> +5V
- R3 pad 2: RS485-3-A -> Net-(D2-Pad2)
- R4 pad 1: Net-(D1-Pad2) -> Net-(R4-Pad1)
- R4 pad 2: 12V_Fused -> D2
- R5 pad 1: Net-(D2-Pad2) -> Net-(R5-Pad1)
- R5 pad 2: /12V_2_Fused -> USB_TXD
- R6 pad 1: Net-(D3-Pad2) -> Net-(R6-Pad1)
- R6 pad 2: /12V_3_Fused -> USB_RXD
Routing:
- net +5V: track 192.1 -> 0.00 mm, vias 1 -> 0
- net 12V_Fused: track 82.9 -> 0.00 mm
- net MEGA_D2: track 71.0 -> 0.00 mm, vias 6 -> 0
- net MEGA_D19: track 66.9 -> 0.00 mm, vias 4 -> 0
- net MEGA_D18: track 59.7 -> 0.00 mm, vias 4 -> 0
- net MEGA_D17: track 48.9 -> 0.00 mm, vias 2 -> 0
- net MEGA_D3: track 46.2 -> 0.00 mm, vias 4 -> 0
- net MEGA_D16: track 39.7 -> 0.00 mm, vias 2 -> 0
- net MEGA_D15: track 22.0 -> 0.00 mm, vias 1 -> 0
- net MEGA_D4: track 21.8 -> 0.00 mm, vias 1 -> 0
- net RS485-3-A: track 21.1 -> 0.00 mm
- net RS485-2-A: track 21.1 -> 0.00 mm
- net RS485-1-A: track 21.0 -> 0.00 mm
- net RS485-3-B: track 20.1 -> 0.00 mm
- net RS485-2-B: track 19.8 -> 0.00 mm
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- removed copper zone on F.Cu, net +12V_2
- removed copper zone on F.Cu, net +12V_3
- removed copper zone on F.Cu, net /12V_2_Fused
- removed copper zone on F.Cu, net /12V_3_Fused
- removed copper zone on F.Cu, net 12V_Fused
- removed copper zone on B.Cu, net GND
- removed copper zone on F.Cu, net GND
- removed copper zone on F.Cu, net Net-(F4-Pad1)
Other:
- board size 82.8 x 55.2 mm -> 94.1 x 58.5 mm
- board text added: "${TITLE} Rev. ${REVISION}"
- board text added: "150MM →"
- board text added: "51.5MM"
- board text added: "87MM"
- board text added: "BRRRRRRRRT"
- board text added: "M3"
- board text added: "← 73MM"
- board text removed: "5V"
- board text removed: "5V POWER"
- board text removed: "BRRRRRRRRRRT"
- board text removed: "BUS 1 POWER"
- board text removed: "BUS 2 POWER"
- board text removed: "BUS 3 POWER"
- board text removed: "D14"
- board text removed: "D15"
- board text removed: "D16"
- board text removed: "D17"
- board text removed: "D18"
- board text removed: "D19"
- board text removed: "D2"
- board text removed: "D3"
- board text removed: "D4"
- board text removed: "GND"
- board text removed: "RS485 Tripe Master Rev. 1"
- board text removed: "VIN"

Commit message: Master WIP
Parts:
- removed R4: 1K, Resistor_SMD:R_0805_2012Metric
- removed SW2: SW_DIP_x01, A10 KiCad Libraries:SW-SMD_DSHP02TSGER
- added Ge: LOGO, LOGO, B.Cu at (91.8, 87.0)
- R10, R12, R14, R5, R6, R7, R8: footprint Resistor_SMD:R_0805_2012Metric -> Resistor_SMD:R_0402_1005Metric
- R2: renamed from R3; footprint Resistor_SMD:R_0805_2012Metric -> Resistor_SMD:R_0402_1005Metric
- R3: renamed from R2; footprint Resistor_SMD:R_0805_2012Metric -> Resistor_SMD:R_0402_1005Metric
- moved U18 128.6 mm to (135.1, 113.9), turned to -90 degrees
- moved F8 128.0 mm to (123.9, 106.7), turned to 90 degrees
- moved U20 127.1 mm to (117.9, 110.2)
- moved F9 122.6 mm to (123.9, 113.9), turned to 90 degrees
- moved J1 121.1 mm to (104.6, 113.5), turned to -90 degrees
- moved J2 118.3 mm to (108.3, 111.2)
- moved D11 117.4 mm to (151.4, 104.2), turned to 90 degrees
- moved U21 116.8 mm to (135.1, 106.4), turned to -90 degrees
- moved C8 116.5 mm to (105.3, 109.2)
- moved D10 116.0 mm to (128.4, 110.2), turned to 180 degrees
- moved C7 115.9 mm to (105.3, 111.2), turned to 180 degrees
- moved C19 115.3 mm to (116.5, 104.5)
- moved R13 114.2 mm to (123.9, 110.2), turned to -90 degrees
- moved PSU3 112.9 mm to (165.0, 110.2), turned to 90 degrees
- moved C2 112.5 mm to (97.6, 109.2)
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Connections:
- BUS3 pad 7: RS485-2- -> RS485-3-
- BUS3 pad 8: RS485-2+ -> RS485-3+
- U18 pad 1: RS485-2+ -> RS485-3+
- U2 pad 26: unconnected-(U2-Pad26) -> D13
- U21 pad 2: RS485-2- -> RS485-3-
Routing:
- net +5V: track 0.00 -> 27.0 mm
- net Net-(BUS2-Pad1): track 0.00 -> 13.5 mm
- net Net-(BUS1-Pad1): track 0.00 -> 13.5 mm
- net Net-(BUS3-Pad1): track 0.00 -> 13.5 mm
- net RS485-3-: track 0.00 -> 13.1 mm
- net RS485-2-: track 0.00 -> 13.1 mm
- net RS485-1-: track 0.00 -> 13.1 mm
- net Net-(F9-Pad2): track 0.00 -> 12.8 mm
- net Net-(F6-Pad2): track 0.00 -> 12.8 mm
- net Net-(F3-Pad2): track 0.00 -> 12.8 mm
- net RS485-2+: track 0.00 -> 12.2 mm
- net RS485-1+: track 0.00 -> 12.2 mm
- net RS485-3+: track 0.00 -> 12.2 mm
- net Net-(F8-Pad1): track 0.00 -> 12.1 mm
- net Net-(F5-Pad1): track 0.00 -> 12.1 mm
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- added copper zone on B.Cu, net GND
- added copper zone on F.Cu, net GND
- added copper zone on B.Cu, net Net-(BUS1-Pad1)
- added copper zone on F.Cu, net Net-(BUS1-Pad1)
- added copper zone on B.Cu, net Net-(BUS2-Pad1)
- added copper zone on F.Cu, net Net-(BUS2-Pad1)
- added copper zone on B.Cu, net Net-(BUS3-Pad1)
- added copper zone on F.Cu, net Net-(BUS3-Pad1)
- added copper zone on B.Cu, net Net-(F10-Pad1)
- added copper zone on F.Cu, net Net-(F10-Pad1)
- added copper zone on B.Cu, net Net-(F4-Pad1)
- added copper zone on F.Cu, net Net-(F4-Pad1)
- added copper zone on B.Cu, net Net-(F7-Pad1)
- added copper zone on F.Cu, net Net-(F7-Pad1)
Other:
- board text added: "${TITLE}"
- board text added: "DCSBIOSKit.com"
- board text added: "Rev. ${REVISION}"
- board text removed: "${TITLE} Rev. ${REVISION}"
- board text removed: "WarthogAtHome.com"

Commit message: Master Rev. 1
Parts:
- removed J1: Conn_01x06_Female, Connector_PinSocket_2.54mm:PinSocket_1x06_P2.54mm_Vertical
- removed U10, U11, U16, U17, U4, U5: TBU-CA065-200-WH, A10 KiCad Libraries:DIO-SMD_3P-L6.5-W4.0-BI
- removed U12, U15, U18, U21, U6, U9: TISP4240M3BJR-S, A10 KiCad Libraries:DO-214AA_L4.4-W3.6-LS5.3-BI
- added G***: LOGO, LOGO, F.Cu at (126.1, 119.0)
- added G***: LOGO, LOGO, B.Cu at (132.2, 92.6)
- added REF**: Tooling Hole, A10 KiCad Libraries:Tooling Hole, F.Cu at (165.0, 68.2)
- added REF**: Tooling Hole, A10 KiCad Libraries:Tooling Hole, F.Cu at (103.2, 121.5)
- F10, F4, F7: footprint A10 KiCad Libraries:FUSE_BK-6013 -> A10 KiCad Libraries:FUSE-TH_XF-506P
- moved H4 131.5 mm to (168.8, 119.6)
- moved H3 116.2 mm to (99.8, 119.6)
- moved H1 50.4 mm to (99.8, 69.6)
- moved C6 29.4 mm to (120.9, 100.5), turned to -90 degrees
- moved D5 27.2 mm to (127.9, 68.5)
- moved C2 26.7 mm to (114.8, 88.9), turned to 180 degrees
- moved C7 26.2 mm to (99.1, 85.7), turned to 90 degrees
- moved D4 24.4 mm to (121.9, 68.5)
- moved R8 23.6 mm to (126.4, 70.2), turned to 180 degrees
- moved C15 22.9 mm to (112.1, 108.9), turned to 90 degrees
- moved R7 21.1 mm to (120.1, 70.2), turned to 180 degrees
- moved Y1 20.5 mm to (109.1, 108.9), turned to 180 degrees
- moved C8 20.4 mm to (106.9, 88.9), turned to 180 degrees
- moved C16 19.7 mm to (106.1, 108.9), turned to 90 degrees
- moved Ge 18.4 mm to (107.2, 97.0)
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Connections:
- D10 pad 1: Net-(D10-Pad1) -> RS485-3+
- D10 pad 2: Net-(D10-Pad2) -> RS485-3-
- D6 pad 1: Net-(D6-Pad1) -> RS485-1+
- D6 pad 2: Net-(D6-Pad2) -> RS485-1-
- D8 pad 1: Net-(D8-Pad1) -> RS485-2+
- D8 pad 2: Net-(D8-Pad2) -> RS485-2-
- F2 pad 2: Net-(D6-Pad2) -> RS485-1-
- F3 pad 1: Net-(D6-Pad1) -> RS485-1+
- F5 pad 2: Net-(D8-Pad2) -> RS485-2-
- F6 pad 1: Net-(D8-Pad1) -> RS485-2+
- F8 pad 2: Net-(D10-Pad2) -> RS485-3-
- F9 pad 1: Net-(D10-Pad1) -> RS485-3+
Routing:
- net +5V: track 27.0 -> 188.2 mm, vias 0 -> 1
- net RESET: track 0.00 -> 104.2 mm, vias 0 -> 6
- net USB_RXD: track 0.00 -> 54.5 mm, vias 0 -> 2
- net USB_TXD: track 0.00 -> 50.0 mm, vias 0 -> 4
- net D19: track 7.99 -> 45.0 mm, vias 0 -> 4
- net D4: track 10.4 -> 46.1 mm, vias 0 -> 6
- net D52: track 0.00 -> 34.5 mm
- net D2: track 10.4 -> 43.8 mm, vias 0 -> 4
- net D18: track 7.47 -> 37.5 mm, vias 0 -> 4
- net D51: track 0.00 -> 29.3 mm, vias 0 -> 2
- net D16: track 7.47 -> 36.4 mm, vias 0 -> 3
- net D50: track 0.00 -> 27.3 mm
- net D17: track 7.99 -> 33.7 mm, vias 0 -> 2
- net D14: track 7.47 -> 26.9 mm, vias 0 -> 4
- net D3: track 10.4 -> 29.7 mm, vias 0 -> 2
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Other:
- board size 94.1 x 58.5 mm -> 75.4 x 56.3 mm
- board text added: "50MM→"
- board text added: "69MM→"
- board text added: "WARNING! DO NOT HOTPLUG!"
- board text removed: "51.5MM"
- board text removed: "87MM"
- board text removed: "BRRRRRRRRT"
